File: Connectors.kicad_sch (KiCad schematic)
At the start: 18 parts, among them J1 MSIM-11-C, J2 USB_B, J3 DM3AT-SF-PEJM5_41_, J4 6437288-4, J5 6437288-4, J7 Conn_ARM_SWD_TagConnect_TC2030

Commit message: routed more sheets, improved analogs. next 5v /analog ground
Parts:
- removed C51, C53: 100nF, Capacitor_SMD:C_0603_1608Metric_Pad1.08x0.95mm_HandSolder, symbol Device:C
- removed C54: 10uF, Capacitor_SMD:C_0603_1608Metric_Pad1.08x0.95mm_HandSolder, symbol Device:C
- removed D10, D11, D12, D13: LED, LED_SMD:LED_0603_1608Metric_Pad1.05x0.95mm_HandSolder, symbol Device:LED
- removed J1: MSIM-11-C, MSIM11C, symbol 0_SamacSys_Parts:MSIM-11-C
- removed J2: USB_B, Connector_USB:USB_B_Lumberg_2411_02_Horizontal, symbol Connector:USB_B
- removed J3: DM3AT-SF-PEJM5_41_, DM3ATSFPEJM541, symbol 0_SamacSys_Parts:DM3AT-SF-PEJM5_41_
- removed J4, J5: 6437288-4, 64372884, symbol 0_SamacSys_Parts:6437288-4
- removed J7: Conn_ARM_SWD_TagConnect_TC2030, Connector:Tag-Connect_TC2030-IDC-FP_2x03_P1.27mm_Vertical, symbol Connector:Conn_ARM_SWD_TagConnect_TC2030
- removed R41: 10R, Resistor_SMD:R_0603_1608Metric_Pad0.98x0.95mm_HandSolder, symbol Device:R
- removed R42, R44, R45: 260R, Resistor_SMD:R_0603_1608Metric_Pad0.98x0.95mm_HandSolder, symbol Device:R
- removed R43: 2k, Resistor_SMD:R_0603_1608Metric_Pad0.98x0.95mm_HandSolder, symbol Device:R
Connections:
- no-connect marks 1 -> 0
