File: CARD_SD.kicad_sch (KiCad schematic)
At the start: 6 parts, among them J8 GSD09002SEU

Commit message: added 3.3v gpio input protection
Other:
- moved on the sheet: C52, C55, J8, R40, R41, R46

Commit message: finished initial esp routing
Changed lines of the file:
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@@
 	(generator_version "9.0")
 	(paper "A5")
-	(rectangle
-		(start 46.99 30.48)
-		(end 182.88 80.01)
-		(stroke
-			(width 0)
-			(type default)
-		)
-		(fill
-			(type none)
-		)
-	)
 	(text_box "Micro SD\nStorage"
 		(exclude_from_sim no)
-		(at 46.99 30.48 0)
+		(at 90.17 104.14 0)
 		(size 12.7 6.35)
 		(margins 0.9525 0.9525 0.9525 0.9525)

Commit message: redid annotations, added test point
Parts:
- renumbered C55 to C41, C52 to C42, J8 to J5, R40 to R29, R46 to R33, R41 to R34
Changed lines of the file:
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@@
 		(on_board yes)
 		(dnp no)
-		(property "Reference" "R41"
+		(property "Reference" "R34"
 			(at 158.496 43.18 0)
 			(effects
@@
 			(project "NCU"
 				(path "/3aee14c3-5480-4f7c-989e-3fef81779034/59880cb1-7ec0-4ddb-9063-a30a9ec86eac"
-					(reference "R41")
+					(reference "R34")
 					(unit 1)
 				)
@@
 		(on_board yes)
 		(dnp no)
-		(property "Reference" "#PWR0109"
+		(property "Reference" "#PWR0186"
 			(at 64.77 76.2 0)
 			(effects
@@
 			(project "NCU"
 				(path "/3aee14c3-5480-4f7c-989e-3fef81779034/59880cb1-7ec0-4ddb-9063-a30a9ec86eac"
-					(reference "#PWR0109")
+					(reference "#PWR0186")
 					(unit 1)
 				)
@@
 		(on_board yes)
 		(dnp no)
-		(property "Reference" "#PWR088"
+		(property "Reference" "#PWR0192"
 			(at 154.94 43.18 0)
 			(effects
@@
 			(project "NCU"
 				(path "/3aee14c3-5480-4f7c-989e-3fef81779034/59880cb1-7ec0-4ddb-9063-a30a9ec86eac"
-					(reference "#PWR088")
+					(reference "#PWR0192")
 					(unit 1)
 				)
@@
 		(on_board yes)
 		(dnp no)
-		(property "Reference" "#PWR0113"
+		(property "Reference" "#PWR0190"
 			(at 146.05 43.18 0)
 			(effects
@@
 			(project "NCU"
 				(path "/3aee14c3-5480-4f7c-989e-3fef81779034/59880cb1-7ec0-4ddb-9063-a30a9ec86eac"
-					(reference "#PWR0113")
+					(reference "#PWR0190")
 					(unit 1)
 				)
@@
 		(on_board yes)
 		(dnp no)
-		(property "Reference" "#PWR0112"
+		(property "Reference" "#PWR0191"
 			(at 147.32 76.2 0)
 			(effects
@@
 			(project "NCU"
 				(path "/3aee14c3-5480-4f7c-989e-3fef81779034/59880cb1-7ec0-4ddb-9063-a30a9ec86eac"
-					(reference "#PWR0112")
+					(reference "#PWR0191")
 					(unit 1)
 				)
@@
 		(on_board yes)
 		(dnp no)
-		(property "Reference" "#PWR0100"
+		(property "Reference" "#PWR0182"
 			(at 26.67 27.94 0)
 			(effects
@@
 			(project "NCU"
 				(path "/3aee14c3-5480-4f7c-989e-3fef81779034/59880cb1-7ec0-4ddb-9063-a30a9ec86eac"
-					(reference "#PWR0100")
+					(reference "#PWR0182")
 					(unit 1)
 				)
@@
 		(on_board yes)
 		(dnp no)
-		(property "Reference" "R40"
+		(property "Reference" "R29"
 			(at 68.072 50.038 0)
 			(effects
@@
 			(project "NCU"
 				(path "/3aee14c3-5480-4f7c-989e-3fef81779034/59880cb1-7ec0-4ddb-9063-a30a9ec86eac"
-					(reference "R40")
+					(reference "R29")
 					(unit 1)
 				)
@@
 		(dnp no)
 		(fields_autoplaced yes)
-		(property "Reference" "J8"
+		(property "Reference" "J5"
 			(at 120.65 41.91 0)
 			(effects
@@
 			(project "NCU"
 				(path "/3aee14c3-5480-4f7c-989e-3fef81779034/59880cb1-7ec0-4ddb-9063-a30a9ec86eac"
-					(reference "J8")
+					(reference "J5")
 					(unit 1)
 				)
@@
 		(on_board yes)
 		(dnp no)
-		(property "Reference" "#PWR099"
+		(property "Reference" "#PWR0183"
 			(at 26.67 35.56 0)
 			(effects
@@
 			(project "NCU"
 				(path "/3aee14c3-5480-4f7c-989e-3fef81779034/59880cb1-7ec0-4ddb-9063-a30a9ec86eac"
-					(reference "#PWR099")
+					(reference "#PWR0183")
 					(unit 1)
 				)
@@
 		(on_board yes)
 		(dnp no)
-		(property "Reference" "#PWR0111"
+		(property "Reference" "#PWR0188"
 			(at 93.98 76.2 0)
 			(effects
@@
 			(project "NCU"
 				(path "/3aee14c3-5480-4f7c-989e-3fef81779034/59880cb1-7ec0-4ddb-9063-a30a9ec86eac"
-					(reference "#PWR0111")
+					(reference "#PWR0188")
 					(unit 1)
 				)
@@
 		(on_board yes)
 		(dnp no)
-		(property "Reference" "C55"
+		(property "Reference" "C41"
 			(at 61.468 61.214 0)
 			(effects
@@
 			(project "NCU"
 				(path "/3aee14c3-5480-4f7c-989e-3fef81779034/59880cb1-7ec0-4ddb-9063-a30a9ec86eac"
-					(reference "C55")
+					(reference "C41")
 					(unit 1)
 				)
@@
 		(on_board yes)
 		(dnp no)
-		(property "Reference" "#PWR0110"
+		(property "Reference" "#PWR0185"
 			(at 64.77 49.53 0)
 			(effects
@@
 			(project "NCU"
 				(path "/3aee14c3-5480-4f7c-989e-3fef81779034/59880cb1-7ec0-4ddb-9063-a30a9ec86eac"
-					(reference "#PWR0110")
+					(reference "#PWR0185")
 					(unit 1)
 				)
@@
 		(on_board yes)
 		(dnp no)
-		(property "Reference" "C52"
+		(property "Reference" "C42"
 			(at 73.406 60.96 0)
 			(effects
@@
 			(project "NCU"
 				(path "/3aee14c3-5480-4f7c-989e-3fef81779034/59880cb1-7ec0-4ddb-9063-a30a9ec86eac"
-					(reference "C52")
+					(reference "C42")
 					(unit 1)
 				)
@@
 		(on_board yes)
 		(dnp no)
-		(property "Reference" "R46"
+		(property "Reference" "R33"
 			(at 149.606 43.18 0)
 			(effects
@@
 			(project "NCU"
 				(path "/3aee14c3-5480-4f7c-989e-3fef81779034/59880cb1-7ec0-4ddb-9063-a30a9ec86eac"
-					(reference "R46")
-					(unit 1)
-				)
+					(reference "R33")
+					(unit 1)
+				)
