File: HSD.kicad_sch (KiCad schematic)
At the start: 11 parts, among them IC5 VND7E025AJTR

Commit message: redid annotations, added test point
Parts:
- R25: renamed from R69; footprint (none) -> Resistor_SMD:R_0603_1608Metric_Pad0.98x0.95mm_HandSolder
- R26: renamed from R70; footprint (none) -> Resistor_SMD:R_0603_1608Metric_Pad0.98x0.95mm_HandSolder
- renumbered C60 to C37, C61 to C38, D17 to D8, IC5 to IC1, R64 to R20, R65 to R21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
