File: INPUTS.kicad_sch (KiCad schematic)
At the start: 0 parts

Commit message: improved analogs
Other:
- sheet INPUT_20V_0 ports: added GND; removed none
- sheet INPUT_20V_1 ports: added GND; removed none
- sheet INPUT_20V_12V ports: added GND; removed none
- sheet INPUT_20V_2 ports: added GND; removed none
- sheet INPUT_20V_3 ports: added GND; removed none
- sheet INPUT_5V_0 ports: added AGND; removed none
- sheet INPUT_5V_1 ports: added AGND; removed none
- sheet INPUT_5V_2 ports: added AGND; removed none
- sheet INPUT_5V_3 ports: added AGND; removed none

Commit message: updated CAN
Changed lines of the file:
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@@
 		(on_board yes)
 		(dnp no)
-		(fields_autoplaced yes)
 		(property "Reference" "#PWR065"
 			(at 25.4 25.4 0)
@@
 			)
 		)
-		(property "Value" "+12V"
-			(at 25.4 16.51 0)
-			(effects
-				(font
-					(size 1.27 1.27)
-				)
+		(property "Value" "12V"
+			(at 24.384 17.526 0)
+			(effects
+				(font
+					(size 1.27 1.27)
+				)
+				(justify left)
 			)
 		)
@@
 		(on_board yes)
 		(dnp no)
-		(fields_autoplaced yes)
 		(property "Reference" "#PWR072"
 			(at 116.84 82.55 0)
@@
 			)
 		)
-		(property "Value" "+12V"
-			(at 116.84 73.66 0)
-			(effects
-				(font
-					(size 1.27 1.27)
-				)
-			)
-		)
+		(property "Value" "12V"
+			(at 115.824 75.184 0)
+			(effects
+				(font
+					(size 1.27 1.27)
+				)
+				(justify left)
+			)
+		)
