File: LSD.kicad_sch (KiCad schematic)
At the start: 7 parts, among them Q4 STS5DNF60L

Commit message: redid annotations, added test point
Parts:
- R18: renamed from R50; footprint (none) -> Resistor_SMD:R_0603_1608Metric_Pad0.98x0.95mm_HandSolder
- R19: renamed from R51; footprint (none) -> Resistor_SMD:R_0603_1608Metric_Pad0.98x0.95mm_HandSolder
- renumbered D11 to D6, D12 to D7, Q4 to Q1, R44 to R16, R45 to R17
