File: MCUPower.kicad_sch (KiCad schematic)
At the start: 20 parts

Commit message: worked on MII pinout
Changed lines of the file:
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@@
+	)
+	(junction
+		(at 190.5 76.2)
+		(diameter 0)
+		(color 0 0 0 0)
 	)
 	(junction
@@
 	(wire
 		(pts
+			(xy 203.2 73.66) (xy 203.2 76.2)
+		)
+		(stroke
+			(width 0)
+			(type default)
+		)
+	)
+	(wire
+		(pts
 			(xy 25.4 38.1) (xy 31.75 38.1)
 		)
@@
 	(wire
 		(pts
+			(xy 190.5 76.2) (xy 203.2 76.2)
+		)
+		(stroke
+			(width 0)
+			(type default)
+		)
+	)
+	(wire
+		(pts
 			(xy 101.6 76.2) (xy 101.6 78.74)
 		)
@@
 		(effects
 			(font
+				(size 1.27 1.27)
+			)
+			(justify left)
+		)
+	)
+	(hierarchical_label "VREF+"
+		(shape passive)
+		(at 203.2 73.66 90)
+		(effects
+			(font

Commit message: added dip switches to wireless disables
Parts:
- C10, C11, C12, C13, C14, C15, C16, C17, C18, C19, C20, C21, C22, C23, C24, C25, C26, C27, C30, C9: footprint Capacitor_SMD:C_0402_1005Metric_Pad0.74x0.62mm_HandSolder -> Capacitor_SMD:C_0603_1608Metric_Pad1.08x0.95mm_HandSolder

Commit message: working on mcu layout
Parts:
- added C28, C29: 2.2uF, Capacitor_SMD:C_0603_1608Metric_Pad1.08x0.95mm_HandSolder, symbol Device:C
- added C31: 220pF, Capacitor_SMD:C_0603_1608Metric_Pad1.08x0.95mm_HandSolder, symbol Device:C
- added C32, C79: 10uF, Capacitor_SMD:C_0603_1608Metric_Pad1.08x0.95mm_HandSolder, symbol Device:C
- added C77, C78, C81: 100nF, Capacitor_SMD:C_0603_1608Metric_Pad1.08x0.95mm_HandSolder, symbol Device:C
- added C80: 1uF, Capacitor_SMD:C_0603_1608Metric_Pad1.08x0.95mm_HandSolder, symbol Device:C
- added FB1: FCM 1608KF-471T03, Inductor_SMD:L_0603_1608Metric_Pad1.05x0.95mm_HandSolder, symbol Device:FerriteBead
- added L4: VLS3015CX-2R2M-H, VLS3015, symbol 0_SamacSys_Parts:VLS3015CX-2R2M-H
- C27: value 4.7uF -> 10uF
Connections:
- net GND: now also C28.2, C29.2, C31.2, C32.2, C77.2, C78.2, C79.2; no longer C25.2, C30.2
- net VBAT: now also C32.1, C79.1, FB1.1; no longer C25.1, C27.1, C30.1
- new net AGND: C25.2, C30.2, C80.2, C81.2
- new net VCAP: C28.1, C29.1
- new net VDDA: C25.1, C30.1, C80.1, C81.1, FB1.2
- new net VDDLDO: C27.1, C77.1, C78.1, L4.2
- new net VLXSMPS: C31.1, L4.1
Other:
- note added: "AKA VDD_SMPS_IN Input supply to switching converter"
- note added: "AKA VDD_SMPS_OUT Output from switching converter"
- note added: "AKA VFBSD"
- moved on the sheet: C23, C24, C25, C30

Commit message: redid annotations, added test point
Parts:
- renumbered C23 to C12, C12 to C13, C24 to C14, C13 to C15, C14 to C16, C32 to C17, C15 to C18, C79 to C19, C16 to C20, C17 to C21, C18 to C22, C19 to C23, C20 to C24, C21 to C25, C22 to C26, C31 to C27, C25 to C28, C27 to C29, C29 to C30, C30 to C31, C28 to C32, C78 to C33, C80 to C34, C77 to C35, C81 to C36, C9 to C8, C26 to C9, L4 to L1
