File: MOD_WLAN.kicad_sch (KiCad schematic)
At the start: 8 parts, among them IC7 ESP32-C6-WROOM-1-N8, SW2 SW_DIP_x01

Commit message: redid annotations, added test point
Parts:
- SW1: renamed from SW2; footprint (none) -> SamacSys_Parts:DS01254L01BE
- renumbered C4 to C48, C73 to C50, C74 to C51, IC7 to IC2, R11 to R47, R12 to R48, R7 to R49
Changed lines of the file:
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@@
 		(on_board yes)
 		(dnp no)
-		(property "Reference" "R7"
+		(property "Reference" "R49"
 			(at 62.738 67.564 90)
 			(effects
@@
 			(project "NCU"
 				(path "/3aee14c3-5480-4f7c-989e-3fef81779034/0cdbc80d-6682-4488-acea-b93c92a9f88d"
-					(reference "R7")
+					(reference "R49")
 					(unit 1)
 				)
@@
 		(on_board yes)
 		(dnp no)
-		(property "Reference" "#PWR0306"
+		(property "Reference" "#PWR0218"
 			(at 114.3 36.83 0)
 			(effects
@@
 			(project "NCU"
 				(path "/3aee14c3-5480-4f7c-989e-3fef81779034/0cdbc80d-6682-4488-acea-b93c92a9f88d"
-					(reference "#PWR0306")
+					(reference "#PWR0218")
 					(unit 1)
 				)
@@
 		(on_board yes)
 		(dnp no)
-		(property "Reference" "SW2"
+		(property "Reference" "SW1"
 			(at 75.692 36.322 0)
 			(effects
@@
 			)
 		)
-		(property "Footprint" ""
+		(property "Footprint" "SamacSys_Parts:DS01254L01BE"
 			(at 83.82 40.64 0)
 			(effects
@@
 			(project "NCU"
 				(path "/3aee14c3-5480-4f7c-989e-3fef81779034/0cdbc80d-6682-4488-acea-b93c92a9f88d"
-					(reference "SW2")
+					(reference "SW1")
 					(unit 1)
 				)
@@
 		(on_board yes)
 		(dnp no)
-		(property "Reference" "R12"
+		(property "Reference" "R48"
 			(at 65.278 25.4 0)
 			(effects
@@
 			(project "NCU"
 				(path "/3aee14c3-5480-4f7c-989e-3fef81779034/0cdbc80d-6682-4488-acea-b93c92a9f88d"
-					(reference "R12")
+					(reference "R48")
 					(unit 1)
 				)
@@
 		(dnp no)
 		(fields_autoplaced yes)
-		(property "Reference" "#PWR0130"
+		(property "Reference" "#PWR0209"
 			(at 26.67 27.94 0)
 			(effects
@@
 			(project "NCU"
 				(path "/3aee14c3-5480-4f7c-989e-3fef81779034/0cdbc80d-6682-4488-acea-b93c92a9f88d"
-					(reference "#PWR0130")
+					(reference "#PWR0209")
 					(unit 1)
 				)
@@
 		(on_board yes)
 		(dnp no)
-		(property "Reference" "R11"
+		(property "Reference" "R47"
 			(at 53.848 76.2 0)
 			(effects
@@
 			(project "NCU"
 				(path "/3aee14c3-5480-4f7c-989e-3fef81779034/0cdbc80d-6682-4488-acea-b93c92a9f88d"
-					(reference "R11")
+					(reference "R47")
 					(unit 1)
 				)
@@
 		(on_board yes)
 		(dnp no)
-		(property "Reference" "IC7"
+		(property "Reference" "IC2"
 			(at 125.73 39.37 0)
 			(effects
@@
 			(project ""
 				(path "/3aee14c3-5480-4f7c-989e-3fef81779034/0cdbc80d-6682-4488-acea-b93c92a9f88d"
-					(reference "IC7")
+					(reference "IC2")
 					(unit 1)
 				)
@@
 		(on_board yes)
 		(dnp no)
-		(property "Reference" "C4"
+		(property "Reference" "C48"
 			(at 71.12 34.2899 0)
 			(effects
@@
 			(project ""
 				(path "/3aee14c3-5480-4f7c-989e-3fef81779034/0cdbc80d-6682-4488-acea-b93c92a9f88d"
-					(reference "C4")
+					(reference "C48")
 					(unit 1)
 				)
@@
 		(dnp no)
 		(fields_autoplaced yes)
-		(property "Reference" "#PWR0305"
+		(property "Reference" "#PWR0219"
 			(at 125.73 22.86 0)
 			(effects
@@
 			(project "NCU"
 				(path "/3aee14c3-5480-4f7c-989e-3fef81779034/0cdbc80d-6682-4488-acea-b93c92a9f88d"
-					(reference "#PWR0305")
+					(reference "#PWR0219")
 					(unit 1)
 				)
@@
 		(dnp no)
 		(fields_autoplaced yes)
-		(property "Reference" "#PWR0303"
+		(property "Reference" "#PWR0213"
 			(at 63.5 25.4 0)
 			(effects
@@
 			(project "NCU"
 				(path "/3aee14c3-5480-4f7c-989e-3fef81779034/0cdbc80d-6682-4488-acea-b93c92a9f88d"
-					(reference "#PWR0303")
+					(reference "#PWR0213")
 					(unit 1)
 				)
@@
 		(dnp no)
 		(fields_autoplaced yes)
-		(property "Reference" "#PWR0300"
+		(property "Reference" "#PWR0220"
 			(at 143.51 99.06 0)
 			(effects
@@
 			(project "NCU"
 				(path "/3aee14c3-5480-4f7c-989e-3fef81779034/0cdbc80d-6682-4488-acea-b93c92a9f88d"
-					(reference "#PWR0300")
+					(reference "#PWR0220")
 					(unit 1)
 				)
@@
 		(on_board yes)
 		(dnp no)
-		(property "Reference" "C73"
+		(property "Reference" "C50"
 			(at 117.094 24.13 0)
 			(effects
@@
 			(project "NCU"
 				(path "/3aee14c3-5480-4f7c-989e-3fef81779034/0cdbc80d-6682-4488-acea-b93c92a9f88d"
-					(reference "C73")
+					(reference "C50")
 					(unit 1)
 				)
@@
 		(dnp no)
 		(fields_autoplaced yes)
-		(property "Reference" "#PWR0301"
+		(property "Reference" "#PWR0216"
 			(at 99.06 46.99 0)
 			(effects
@@
 			(project "NCU"
 				(path "/3aee14c3-5480-4f7c-989e-3fef81779034/0cdbc80d-6682-4488-acea-b93c92a9f88d"
-					(reference "#PWR0301")
+					(reference "#PWR0216")
 					(unit 1)
 				)
@@
 		(on_board yes)
 		(dnp no)
-		(property "Reference" "#PWR0304"
+		(property "Reference" "#PWR0214"
 			(at 67.31 49.53 0)
 			(effects
@@
 			(project "NCU"
 				(path "/3aee14c3-5480-4f7c-989e-3fef81779034/0cdbc80d-6682-4488-acea-b93c92a9f88d"
-					(reference "#PWR0304")
+					(reference "#PWR0214")
 					(unit 1)
 				)
@@
 		(dnp no)
 		(fields_autoplaced yes)
-		(property "Reference" "#PWR0302"
+		(property "Reference" "#PWR0212"
 			(at 52.07 59.69 0)
 			(effects
@@
 			(project "NCU"
 				(path "/3aee14c3-5480-4f7c-989e-3fef81779034/0cdbc80d-6682-4488-acea-b93c92a9f88d"
-					(reference "#PWR0302")
+					(reference "#PWR0212")
 					(unit 1)
 				)
@@
 		(dnp no)
 		(fields_autoplaced yes)
-		(property "Reference" "#PWR0131"
+		(property "Reference" "#PWR0211"
 			(at 26.67 35.56 0)
 			(effects
@@
 			(project "NCU"
 				(path "/3aee14c3-5480-4f7c-989e-3fef81779034/0cdbc80d-6682-4488-acea-b93c92a9f88d"
-					(reference "#PWR0131")
+					(reference "#PWR0211")
 					(unit 1)
 				)
@@
 		(on_board yes)
 		(dnp no)
-		(property "Reference" "C74"
+		(property "Reference" "C51"
 			(at 128.524 24.13 0)
 			(effects
@@
 			(project "NCU"
 				(path "/3aee14c3-5480-4f7c-989e-3fef81779034/0cdbc80d-6682-4488-acea-b93c92a9f88d"
-					(reference "C74")
-					(unit 1)
-				)
+					(reference "C51")
+					(unit 1)
+				)
