File: pcb/GPIO.kicad_sch (KiCad schematic)
At the start: 0 parts

Commit message: updated ethernet
Other:
- sheet INPUT_3V3_0 ports: added 3V3; removed none
- sheet INPUT_3V3_1 ports: added 3V3; removed none
- sheet INPUT_3V3_2 ports: added 3V3; removed none
- sheet INPUT_3V3_3 ports: added 3V3; removed none
