File: pcb/MCU.kicad_sch (KiCad schematic)
At the start: 14 parts, among them U4 STM32H745ZITx, Y2 NX3215SA-32.768K-STD-MUS-2, Y3 Crystal_GND24

Commit message: added better lsds
Connections:
- net LSD2_STAT: now reaches U4.57 (PE7)
- net LSD3_STAT: now reaches U4.58 (PE8)
- net LSD0_STAT: now reaches U4.60 (PE10)
- net LSD1_STAT: now reaches U4.62 (PE12)
- no-connect marks 0 -> 24
Changed lines of the file:
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@@
 		(color 0 0 0 0)
 	)
+	(no_connect
+		(at 134.62 121.92)
+	)
+	(no_connect
+		(at 220.98 116.84)
+	)
+	(no_connect
+		(at 134.62 157.48)
+	)
+	(no_connect
+		(at 220.98 187.96)
+	)
+	(no_connect
+		(at 220.98 172.72)
+	)
+	(no_connect
+		(at 134.62 109.22)
+	)
+	(no_connect
+		(at 220.98 223.52)
+	)
+	(no_connect
+		(at 220.98 170.18)
+	)
+	(no_connect
+		(at 134.62 111.76)
+	)
+	(no_connect
+		(at 134.62 116.84)
+	)
+	(no_connect
+		(at 220.98 149.86)
+	)
+	(no_connect
+		(at 134.62 119.38)
+	)
+	(no_connect
+		(at 134.62 187.96)
+	)
+	(no_connect
+		(at 134.62 106.68)
+	)
+	(no_connect
+		(at 220.98 215.9)
+	)
+	(no_connect
+		(at 220.98 220.98)
+	)
+	(no_connect
+		(at 134.62 104.14)
+	)
+	(no_connect
+		(at 134.62 144.78)
+	)
+	(no_connect
+		(at 134.62 114.3)
+	)
+	(no_connect
+		(at 220.98 218.44)
+	)
+	(no_connect
+		(at 220.98 147.32)
+	)
+	(no_connect
+		(at 220.98 121.92)
+	)
+	(no_connect
+		(at 220.98 137.16)
+	)
+	(no_connect
+		(at 134.62 101.6)
+	)
 	(wire
 		(pts
@@
 	(wire
 		(pts
+			(xy 127 175.26) (xy 134.62 175.26)
+		)
+		(stroke
+			(width 0)
+			(type default)
+		)
+	)
+	(wire
+		(pts
 			(xy 170.18 54.61) (xy 170.18 58.42)
 		)
@@
 	(wire
 		(pts
+			(xy 127 170.18) (xy 134.62 170.18)
+		)
+		(stroke
+			(width 0)
+			(type default)
+		)
+	)
+	(wire
+		(pts
 			(xy 228.6 144.78) (xy 220.98 144.78)
 		)
@@
 	(wire
 		(pts
+			(xy 127 167.64) (xy 134.62 167.64)
+		)
+		(stroke
+			(width 0)
+			(type default)
+		)
+	)
+	(wire
+		(pts
 			(xy 355.6 48.26) (xy 355.6 49.53)
 		)
@@
 		(pts
 			(xy 220.98 175.26) (xy 228.6 175.26)
+		)
+		(stroke
+			(width 0)
+			(type default)
+		)
+	)
+	(wire
+		(pts
+			(xy 127 180.34) (xy 134.62 180.34)
 		)
 		(stroke
@@
 		)
 	)
+	(hierarchical_label "LSD1_STAT"
+		(shape passive)
+		(at 127 180.34 180)
+		(effects
+			(font
+				(size 1.27 1.27)
+			)
+			(justify right)
+		)
+	)
 	(hierarchical_label "ETH_TXD0"
 		(shape passive)
@@
 		)
 	)
+	(hierarchical_label "LSD3_STAT"
+		(shape passive)
+		(at 127 170.18 180)
+		(effects
+			(font
+				(size 1.27 1.27)
+			)
+			(justify right)
+		)
+	)
+	(hierarchical_label "LSD0_STAT"
+		(shape passive)
+		(at 127 175.26 180)
+		(effects
+			(font
+				(size 1.27 1.27)
+			)
+			(justify right)
+		)
+	)
 	(hierarchical_label "SD_WP"
 		(shape passive)
@@
 		)
 	)
+	(hierarchical_label "LSD2_STAT"
+		(shape passive)
+		(at 127 167.64 180)
+		(effects
+			(font
+				(size 1.27 1.27)
+			)
+			(justify right)
+		)
+	)

Commit message: power done
Parts:
- added TP10: BOOT, TestPoint:TestPoint_THTPad_D2.0mm_Drill1.0mm, symbol Connector:TestPoint
- added TP11: NRST, TestPoint:TestPoint_THTPad_D2.0mm_Drill1.0mm, symbol Connector:TestPoint
- JP1: footprint Jumper:SolderJumper-2_P1.3mm_Open_TrianglePad1.0x1.5mm -> Jumper:SolderJumper-2_P1.3mm_Open_RoundedPad1.0x1.5mm
Connections:
- net STM_NRST: now also TP11.1
- net at JP1.1 (A), R88.1, U4.135 (BOOT0): now also TP10.1
Changed lines of the file:
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@@
 	)
 	(junction
+		(at 120.65 68.58)
+		(diameter 0)
+		(color 0 0 0 0)
+	)
+	(junction
 		(at 88.9 73.66)
 		(diameter 0)
@@
 	)
 	(junction
+		(at 107.95 73.66)
+		(diameter 0)
+		(color 0 0 0 0)
+	)
+	(junction
 		(at 175.26 250.19)
 		(diameter 0)
@@
 	(wire
 		(pts
+			(xy 107.95 73.66) (xy 134.62 73.66)
+		)
+		(stroke
+			(width 0)
+			(type default)
+		)
+	)
+	(wire
+		(pts
 			(xy 78.74 67.31) (xy 78.74 68.58)
 		)
@@
 	(wire
 		(pts
+			(xy 107.95 63.5) (xy 107.95 73.66)
+		)
+		(stroke
+			(width 0)
+			(type default)
+		)
+	)
+	(wire
+		(pts
 			(xy 187.96 54.61) (xy 187.96 58.42)
 		)
@@
 	(wire
 		(pts
-			(xy 88.9 73.66) (xy 134.62 73.66)
+			(xy 88.9 73.66) (xy 107.95 73.66)
 		)
 		(stroke
@@
 	(wire
 		(pts
+			(xy 120.65 63.5) (xy 120.65 68.58)
+		)
+		(stroke
+			(width 0)
+			(type default)
+		)
+	)
+	(wire
+		(pts
 			(xy 129.54 137.16) (xy 134.62 137.16)
 		)
@@
 	(wire
 		(pts
-			(xy 78.74 68.58) (xy 134.62 68.58)
+			(xy 78.74 68.58) (xy 120.65 68.58)
 		)
 		(stroke
@@
 	(wire
 		(pts
+			(xy 120.65 68.58) (xy 134.62 68.58)
+		)
+		(stroke
+			(width 0)
+			(type default)
+		)
+	)
+	(wire
+		(pts
 			(xy 154.94 54.61) (xy 154.94 58.42)
 		)
@@
 	)
 	(symbol
+		(lib_id "Connector:TestPoint")
+		(at 107.95 63.5 0)
+		(mirror y)
+		(unit 1)
+		(exclude_from_sim no)
+		(in_bom yes)
+		(on_board yes)
+		(dnp no)
+		(property "Reference" "TP10"
+			(at 109.22 59.436 0)
+			(effects
+				(font
+					(size 1.27 1.27)
+				)
+				(justify right)
+			)
+		)
+		(property "Value" "BOOT"
+			(at 109.22 61.468 0)
+			(effects
+				(font
+					(size 1.27 1.27)
+				)
+				(justify right)
+			)
+		)
+		(property "Footprint" "TestPoint:TestPoint_THTPad_D2.0mm_Drill1.0mm"
+			(at 102.87 63.5 0)
+			(effects
+				(font
+					(size 1.27 1.27)
+				)
+				(hide yes)
+			)
+		)
+		(property "Datasheet" "~"
+			(at 102.87 63.5 0)
+			(effects
+				(font
+					(size 1.27 1.27)
+				)
+				(hide yes)
+			)
+		)
+		(property "Description" "test point"
+			(at 107.95 63.5 0)
+			(effects
+				(font
+					(size 1.27 1.27)
+				)
+				(hide yes)
+			)
+		)
+		(pin "1"
+		)
+		(instances
+			(project "NCU"
+				(path "/3aee14c3-5480-4f7c-989e-3fef81779034/d2b1e1a0-8b64-49ff-b975-b40fa2d33dc6"
+					(reference "TP10")
+					(unit 1)
+				)
+			)
+		)
+	)
+	(symbol
 		(lib_id "Device:R")
 		(at 81.28 243.84 0)
@@
 	)
 	(symbol
+		(lib_id "Connector:TestPoint")
+		(at 120.65 63.5 0)
+		(mirror y)
+		(unit 1)
+		(exclude_from_sim no)
+		(in_bom yes)
+		(on_board yes)
+		(dnp no)
+		(property "Reference" "TP11"
+			(at 122.174 59.182 0)
+			(effects
+				(font
+					(size 1.27 1.27)
+				)
+				(justify right)
+			)
+		)
+		(property "Value" "NRST"
+			(at 121.92 61.468 0)
+			(effects
+				(font
+					(size 1.27 1.27)
+				)
+				(justify right)
+			)
+		)
+		(property "Footprint" "TestPoint:TestPoint_THTPad_D2.0mm_Drill1.0mm"
+			(at 115.57 63.5 0)
+			(effects
+				(font
+					(size 1.27 1.27)
+				)
+				(hide yes)
+			)
+		)
+		(property "Datasheet" "~"
+			(at 115.57 63.5 0)
+			(effects
+				(font
+					(size 1.27 1.27)
+				)
+				(hide yes)
+			)
+		)
+		(property "Description" "test point"
+			(at 120.65 63.5 0)
+			(effects
+				(font
+					(size 1.27 1.27)
+				)
+				(hide yes)
+			)
+		)
+		(pin "1"
+		)
+		(instances
+			(project "NCU"
+				(path "/3aee14c3-5480-4f7c-989e-3fef81779034/d2b1e1a0-8b64-49ff-b975-b40fa2d33dc6"
+					(reference "TP11")
+					(unit 1)
+				)
+			)
+		)
+	)
+	(symbol
 		(lib_id "power:GND")
 		(at 342.9 30.48 180)
@@
 			)
 		)
-		(property "Footprint" "Jumper:SolderJumper-2_P1.3mm_Open_TrianglePad1.0x1.5mm"
+		(property "Footprint" "Jumper:SolderJumper-2_P1.3mm_Open_RoundedPad1.0x1.5mm"
 			(at 88.9 63.5 0)
 			(effects

Commit message: reannotated, updated some symbols
Parts:
- added D27: SP0504BAHT, Package_TO_SOT_SMD:SOT-23-5, symbol Power_Protection:SP0504BAHT
- C90: renamed from C83; value 5.6pF -> 8.2pF
- C92: renamed from C85; value 5.6pF -> 8.2pF
- renumbered C82 to C89, C84 to C91, C86 to C93, D27 to D26, JP1 to JP12, R86 to R123, R87 to R124, R88 to R125, R89 to R126, TP10 to TP18, TP11 to TP19, U4 to U7
Connections:
- net GND: now also D27.2 (A)
- net STM_NRST: now also D27.4 (K)
- net STM_SWDCLK: now also D27.3 (K)
- net STM_SWDIO: now also D27.1 (K)
- net STM_SWO: now also D27.5 (K)

Commit message: minor changes before layout
Connections:
- net at R124.1: now also U7.65 (PE15)
- no-connect marks 24 -> 23
Other:
- moved on the sheet: D26, R124
Changed lines of the file:
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@@
 	(generator_version "9.0")
 	(paper "A3")
-	(rectangle
-		(start 45.72 223.52)
-		(end 106.68 271.78)
-		(stroke
-			(width 0)
-			(type default)
-		)
-		(fill
-			(type none)
-		)
-	)
 	(text_box "Solder jumper for boot recovery - bridge to enter system bootloader mode"
 		(exclude_from_sim no)
@@
 		)
 	)
-	(text_box "Status LEDs\nDebug"
-		(exclude_from_sim no)
-		(at 45.72 223.52 0)
-		(size 15.24 6.35)
-		(margins 0.9525 0.9525 0.9525 0.9525)
-		(stroke
-			(width -0.0001)
-			(type solid)
-		)
-		(fill
-			(type none)
-		)
-		(effects
-			(font
-				(face "KiCad Font")
-				(size 1.27 1.27)
-			)
-			(justify left top)
-		)
-	)
 	(junction
 		(at 266.7 101.6)
@@
 	)
 	(no_connect
-		(at 134.62 187.96)
-	)
-	(no_connect
 		(at 134.62 106.68)
 	)
@@
 	(wire
 		(pts
+			(xy 95.25 187.96) (xy 95.25 190.5)
+		)
+		(stroke
+			(width 0)
+			(type default)
+		)
+	)
+	(wire
+		(pts
 			(xy 271.78 111.76) (xy 279.4 111.76)
 		)
@@
 	(wire
 		(pts
-			(xy 81.28 238.76) (xy 81.28 240.03)
-		)
-		(stroke
-			(width 0)
-			(type default)
-		)
-	)
-	(wire
-		(pts
 			(xy 127 177.8) (xy 134.62 177.8)
 		)
@@
 	(wire
 		(pts
+			(xy 95.25 187.96) (xy 134.62 187.96)
+		)
+		(stroke
+			(width 0)
+			(type default)
+		)
+	)
+	(wire
+		(pts
 			(xy 220.98 106.68) (xy 228.6 106.68)
 		)
@@
 	(wire
 		(pts
-			(xy 81.28 247.65) (xy 81.28 248.92)
+			(xy 95.25 198.12) (xy 95.25 199.39)
 		)
 		(stroke
@@
 	(wire
 		(pts
-			(xy 81.28 256.54) (xy 81.28 257.81)
+			(xy 95.25 207.01) (xy 95.25 208.28)
 		)
 		(stroke
@@
 	(symbol
 		(lib_id "Device:R")
-		(at 81.28 243.84 0)
+		(at 95.25 194.31 0)
 		(unit 1)
 		(exclude_from_sim no)
@@
 		(dnp no)
 		(property "Reference" "R124"
-			(at 84.836 242.57 0)
+			(at 98.806 193.04 0)
 			(effects
 				(font
@@
 		)
 		(property "Value" "260R"
-			(at 85.598 244.856 0)
+			(at 99.568 195.326 0)
 			(effects
 				(font
@@
 		)
 		(property "Footprint" "Resistor_SMD:R_0603_1608Metric_Pad0.98x0.95mm_HandSolder"
-			(at 79.502 243.84 90)
+			(at 93.472 194.31 90)
 			(effects
 				(font
@@
 		)
 		(property "Datasheet" "~"
-			(at 81.28 243.84 0)
+			(at 95.25 194.31 0)
 			(effects
 				(font
@@
 		)
 		(property "Description" "Resistor"
-			(at 81.28 243.84 0)
+			(at 95.25 194.31 0)
 			(effects
 				(font
@@
 	(symbol
 		(lib_id "Device:LED")
-		(at 81.28 252.73 90)
+		(at 95.25 203.2 90)
 		(unit 1)
 		(exclude_from_sim no)
@@
 		(dnp no)
 		(property "Reference" "D26"
-			(at 84.582 252.984 90)
+			(at 98.552 203.454 90)
 			(effects
 				(font
@@
 		)
 		(property "Value" "LED"
-			(at 84.582 255.524 90)
+			(at 98.552 205.994 90)
 			(effects
 				(font
@@
 		)
 		(property "Footprint" "LED_SMD:LED_0603_1608Metric_Pad1.05x0.95mm_HandSolder"
-			(at 81.28 252.73 0)
+			(at 95.25 203.2 0)
 			(effects
 				(font
@@
 		)
 		(property "Datasheet" "~"
-			(at 81.28 252.73 0)
+			(at 95.25 203.2 0)
 			(effects
 				(font
@@
 		)
 		(property "Description" "Light emitting diode"
-			(at 81.28 252.73 0)
+			(at 95.25 203.2 0)
 			(effects
 				(font
@@
 		)
 		(property "Sim.Pins" "1=K 2=A"
-			(at 81.28 252.73 0)
+			(at 95.25 203.2 0)
 			(effects
 				(font
@@
 	(symbol
 		(lib_id "power:GND")
-		(at 81.28 257.81 0)
+		(at 95.25 208.28 0)
 		(unit 1)
 		(exclude_from_sim no)
@@
 		(dnp no)
 		(property "Reference" "#PWR0413"
-			(at 81.28 264.16 0)
+			(at 95.25 214.63 0)
 			(effects
 				(font
@@
 		)
 		(property "Value" "GND"
-			(at 81.28 261.874 0)
+			(at 95.25 212.344 0)
 			(effects
 				(font
@@
 		)
 		(property "Footprint" ""
-			(at 81.28 257.81 0)
+			(at 95.25 208.28 0)
 			(effects
 				(font
@@
 		)
 		(property "Datasheet" ""
-			(at 81.28 257.81 0)
+			(at 95.25 208.28 0)
 			(effects
 				(font
@@
 		)
 		(property "Description" "Power symbol creates a global label with name \"GND\" , ground"
-			(at 81.28 257.81 0)
+			(at 95.25 208.28 0)
 			(effects
 				(font

Commit message: initial microcontroller layout
Connections:
- net RCC_OSC32_IN: now also C93.1, Y2.2
- net RCC_OSC32_OUT: now also C91.1, Y2.1
- net RCC_OSC_IN: no longer C93.1, Y2.2
- net RCC_OSC_OUT: no longer C91.1, Y2.1
Changed lines of the file:
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@@
-		)
-	)
-	(label "RCC_OSC_IN"
-		(at 368.3 76.2 180)
-		(effects
-			(font
-				(size 1.27 1.27)
-			)
-			(justify right bottom)
 		)
 	)
@@
 		)
 	)
+	(label "RCC_OSC32_OUT"
+		(at 317.5 76.2 0)
+		(effects
+			(font
+				(size 1.27 1.27)
+			)
+			(justify left bottom)
+		)
+	)
 	(label "VCAP"
 		(at 127 43.18 0)
@@
 			)
 			(justify left bottom)
+		)
+	)
+	(label "RCC_OSC32_IN"
+		(at 368.3 76.2 180)
+		(effects
+			(font
+				(size 1.27 1.27)
+			)
+			(justify right bottom)
 		)
 	)
@@
 		(effects
 			(font
-				(size 1.27 1.27)
-			)
-			(justify left bottom)
-		)
-	)
-	(label "RCC_OSC_OUT"
-		(at 317.5 76.2 0)
-		(effects
-			(font

Commit message: sd card slot initial attempt (I meant SIM before)
Connections:
- net SD_WP: no longer names the net of U7.97 (PA8)
- no-connect marks 23 -> 24
Changed lines of the file:
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@@
+	)
+	(no_connect
+		(at 220.98 88.9)
 	)
 	(no_connect
@@
 	(wire
 		(pts
-			(xy 220.98 88.9) (xy 228.6 88.9)
-		)
-		(stroke
-			(width 0)
-			(type default)
-		)
-	)
-	(wire
-		(pts
 			(xy 228.6 157.48) (xy 220.98 157.48)
 		)
@@
 		)
 	)
-	(hierarchical_label "SD_WP"
-		(shape passive)
-		(at 228.6 88.9 0)
-		(effects
-			(font
-				(size 1.27 1.27)
-			)
-			(justify left)
-		)
-	)

Commit message: routed LSDs to micro
Parts:
- removed TP19: NRST, TestPoint:TestPoint_THTPad_D2.0mm_Drill1.0mm, symbol Connector:TestPoint
Changed lines of the file:
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@@
 	)
 	(junction
-		(at 120.65 68.58)
-		(diameter 0)
-		(color 0 0 0 0)
-	)
-	(junction
 		(at 88.9 73.66)
 		(diameter 0)
@@
 	(wire
 		(pts
-			(xy 120.65 63.5) (xy 120.65 68.58)
-		)
-		(stroke
-			(width 0)
-			(type default)
-		)
-	)
-	(wire
-		(pts
 			(xy 266.7 101.6) (xy 279.4 101.6)
 		)
@@
 	(wire
 		(pts
-			(xy 78.74 68.58) (xy 120.65 68.58)
+			(xy 78.74 68.58) (xy 134.62 68.58)
 		)
 		(stroke
@@
 	(wire
 		(pts
-			(xy 120.65 68.58) (xy 134.62 68.58)
-		)
-		(stroke
-			(width 0)
-			(type default)
-		)
-	)
-	(wire
-		(pts
 			(xy 154.94 54.61) (xy 154.94 58.42)
 		)
@@
 					(unit 1)
 				)
-			)
-		)
-	)
-	(symbol
-		(lib_id "Connector:TestPoint")
-		(at 120.65 63.5 0)
-		(mirror y)
-		(unit 1)
-		(exclude_from_sim no)
-		(in_bom yes)
-		(on_board yes)
-		(dnp no)
-		(property "Reference" "TP19"
-			(at 122.174 59.182 0)
-			(effects
-				(font
-					(size 1.27 1.27)
-				)
-				(justify right)
-			)
-		)
-		(property "Value" "NRST"
-			(at 121.92 61.468 0)
-			(effects
-				(font
-					(size 1.27 1.27)
-				)
-				(justify right)
-			)
-		)
-		(property "Footprint" "TestPoint:TestPoint_THTPad_D2.0mm_Drill1.0mm"
-			(at 115.57 63.5 0)
-			(effects
-				(font
-					(size 1.27 1.27)
-				)
-				(hide yes)
-			)
-		)
-		(property "Datasheet" "~"
-			(at 115.57 63.5 0)
-			(effects
-				(font
-					(size 1.27 1.27)
-				)
-				(hide yes)
-			)
-		)
-		(property "Description" "test point"
-			(at 120.65 63.5 0)
-			(effects
-				(font
-					(size 1.27 1.27)
-				)
-				(hide yes)
-			)
-		)
-		(pin "1"
-		)
-		(instances
-			(project "NCU"
-				(path "/3aee14c3-5480-4f7c-989e-3fef81779034/d2b1e1a0-8b64-49ff-b975-b40fa2d33dc6"
-					(reference "TP19")
-					(unit 1)
-				)

Commit message: removed AGND and added ground garden
Connections:
- net AGND is gone; now on net GND: U7.34 (VSSA)
Other:
- sheet MCU Power ports: added none; removed AGND
