File: pcb/MCU.kicad_sch (KiCad schematic)
At the start: 16 parts, among them U7 STM32H745ZITx, Y2 NX3215SA-32.768K-STD-MUS-2, Y3 Crystal_GND24

Commit message: added 10k resistor to USB VBUS line
Parts:
- added R46: 10k, Resistor_SMD:R_0603_1608Metric_Pad0.98x0.95mm_HandSolder, symbol Device:R
Connections:
- net USB_VBUS: now also R46.2; no longer U7.98 (PA9)
- new net: R46.1, U7.98 (PA9)
Changed lines of the file:
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@@
 	(wire
 		(pts
-			(xy 228.6 91.44) (xy 220.98 91.44)
+			(xy 233.68 91.44) (xy 231.14 91.44)
 		)
 		(stroke
@@
 		(pts
 			(xy 228.6 127) (xy 220.98 127)
+		)
+		(stroke
+			(width 0)
+			(type default)
+		)
+	)
+	(wire
+		(pts
+			(xy 223.52 91.44) (xy 220.98 91.44)
 		)
 		(stroke
@@
 	(hierarchical_label "USB_VBUS"
 		(shape passive)
-		(at 228.6 91.44 0)
+		(at 233.68 91.44 0)
 		(effects
 			(font
@@
 					(unit 1)
 				)
+			)
+		)
+	)
+	(symbol
+		(lib_id "Device:R")
+		(at 227.33 91.44 90)
+		(unit 1)
+		(exclude_from_sim no)
+		(in_bom yes)
+		(on_board yes)
+		(dnp no)
+		(property "Reference" "R46"
+			(at 225.552 88.9 90)
+			(effects
+				(font
+					(size 1.27 1.27)
+				)
+			)
+		)
+		(property "Value" "10k"
+			(at 229.616 88.9 90)
+			(effects
+				(font
+					(size 1.27 1.27)
+				)
+			)
+		)
+		(property "Footprint" "Resistor_SMD:R_0603_1608Metric_Pad0.98x0.95mm_HandSolder"
+			(at 227.33 93.218 90)
+			(effects
+				(font
+					(size 1.27 1.27)
+				)
+				(hide yes)
+			)
+		)
+		(property "Datasheet" "~"
+			(at 227.33 91.44 0)
+			(effects
+				(font
+					(size 1.27 1.27)
+				)
+				(hide yes)
+			)
+		)
+		(property "Description" "Resistor"
+			(at 227.33 91.44 0)
+			(effects
+				(font
+					(size 1.27 1.27)
+				)
+				(hide yes)
+			)
+		)
+		(pin "1"
+		)
+		(pin "2"
+		)
+		(instances
+			(project "NCU"
+				(path "/3aee14c3-5480-4f7c-989e-3fef81779034/d2b1e1a0-8b64-49ff-b975-b40fa2d33dc6"
+					(reference "R46")
+					(unit 1)
+				)

Commit message: updates from bom release
Parts:
- C89: value 100nF -> 100n
- C90, C92: value 8.2pF -> 8.2p
- C91, C93: value 5.1pF -> 5.1p
- R124: value 260R -> 620
Changed lines of the file:
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@@
 			)
 		)
-		(property "Value" "260R"
+		(property "Value" "620"
 			(at 99.568 195.326 0)
 			(effects
@@
 			)
 		)
-		(property "Value" "5.1pF"
+		(property "Value" "5.1p"
 			(at 358.14 83.82 0)
 			(effects
@@
 			)
 		)
-		(property "Value" "5.1pF"
+		(property "Value" "5.1p"
 			(at 332.74 83.82 0)
 			(effects
@@
 			)
 		)
-		(property "Value" "100nF"
+		(property "Value" "100n"
 			(at 78.74 74.93 0)
 			(effects
@@
 			)
 		)
-		(property "Value" "8.2pF"
+		(property "Value" "8.2p"
 			(at 332.74 45.72 0)
 			(effects
@@
 			)
 		)
-		(property "Value" "8.2pF"
+		(property "Value" "8.2p"
 			(at 358.14 45.72 0)
 			(effects

Commit message: updated to match board changes
Parts:
- D27: now not fitted
Changed lines of the file:
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@@
 		(in_bom yes)
 		(on_board yes)
-		(dnp no)
+		(dnp yes)
 		(fields_autoplaced yes)
 		(property "Reference" "D27"
