File: pcb/CAN_BUS.kicad_sch (KiCad schematic)
At the start: 4 parts, among them U2 SN65HVD230

Commit message: added better lsds
Parts:
- added R90: 120R, Resistor_SMD:R_0603_1608Metric_Pad0.98x0.95mm_HandSolder, symbol Device:R
Connections:
- net HI: now also R90.1
- net LO: now also R90.2
Changed lines of the file:
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@@
 	)
 	(junction
-		(at 85.09 58.42)
+		(at 57.15 60.96)
 		(diameter 0)
 		(color 0 0 0 0)
@@
 	)
 	(junction
+		(at 85.09 60.96)
+		(diameter 0)
+		(color 0 0 0 0)
+	)
+	(junction
 		(at 101.6 66.04)
+		(diameter 0)
+		(color 0 0 0 0)
+	)
+	(junction
+		(at 57.15 53.34)
 		(diameter 0)
 		(color 0 0 0 0)
@@
 	)
 	(junction
-		(at 82.55 55.88)
+		(at 82.55 53.34)
 		(diameter 0)
 		(color 0 0 0 0)
@@
 	(wire
 		(pts
-			(xy 78.74 55.88) (xy 82.55 55.88)
+			(xy 50.8 53.34) (xy 57.15 53.34)
 		)
 		(stroke
@@
 	(wire
 		(pts
-			(xy 82.55 55.88) (xy 82.55 86.36)
+			(xy 82.55 53.34) (xy 82.55 86.36)
+		)
+		(stroke
+			(width 0)
+			(type default)
+		)
+	)
+	(wire
+		(pts
+			(xy 88.9 53.34) (xy 88.9 55.88)
 		)
 		(stroke
@@
 	(wire
 		(pts
+			(xy 88.9 60.96) (xy 88.9 58.42)
+		)
+		(stroke
+			(width 0)
+			(type default)
+		)
+	)
+	(wire
+		(pts
 			(xy 111.76 60.96) (xy 111.76 66.04)
 		)
@@
 	(wire
 		(pts
-			(xy 85.09 58.42) (xy 91.44 58.42)
+			(xy 85.09 60.96) (xy 88.9 60.96)
 		)
 		(stroke
@@
 	(wire
 		(pts
+			(xy 88.9 58.42) (xy 91.44 58.42)
+		)
+		(stroke
+			(width 0)
+			(type default)
+		)
+	)
+	(wire
+		(pts
+			(xy 57.15 53.34) (xy 82.55 53.34)
+		)
+		(stroke
+			(width 0)
+			(type default)
+		)
+	)
+	(wire
+		(pts
 			(xy 26.67 25.4) (xy 26.67 26.67)
 		)
@@
 	(wire
 		(pts
-			(xy 78.74 58.42) (xy 85.09 58.42)
-		)
-		(stroke
-			(width 0)
-			(type default)
-		)
-	)
-	(wire
-		(pts
-			(xy 85.09 58.42) (xy 85.09 83.82)
-		)
-		(stroke
-			(width 0)
-			(type default)
-		)
-	)
-	(wire
-		(pts
-			(xy 82.55 55.88) (xy 91.44 55.88)
+			(xy 85.09 60.96) (xy 85.09 83.82)
+		)
+		(stroke
+			(width 0)
+			(type default)
+		)
+	)
+	(wire
+		(pts
+			(xy 50.8 60.96) (xy 57.15 60.96)
+		)
+		(stroke
+			(width 0)
+			(type default)
+		)
+	)
+	(wire
+		(pts
+			(xy 88.9 55.88) (xy 91.44 55.88)
+		)
+		(stroke
+			(width 0)
+			(type default)
+		)
+	)
+	(wire
+		(pts
+			(xy 57.15 60.96) (xy 85.09 60.96)
+		)
+		(stroke
+			(width 0)
+			(type default)
+		)
+	)
+	(wire
+		(pts
+			(xy 82.55 53.34) (xy 88.9 53.34)
 		)
 		(stroke
@@
 	(hierarchical_label "LO"
 		(shape passive)
-		(at 78.74 58.42 180)
+		(at 50.8 60.96 180)
 		(effects
 			(font
@@
 	(hierarchical_label "HI"
 		(shape passive)
-		(at 78.74 55.88 180)
+		(at 50.8 53.34 180)
 		(effects
 			(font
@@
 					(unit 1)
 				)
+			)
+		)
+	)
+	(symbol
+		(lib_id "Device:R")
+		(at 57.15 57.15 0)
+		(unit 1)
+		(exclude_from_sim no)
+		(in_bom no)
+		(on_board yes)
+		(dnp yes)
+		(fields_autoplaced yes)
+		(property "Reference" "R90"
+			(at 59.69 55.8799 0)
+			(effects
+				(font
+					(size 1.27 1.27)
+				)
+				(justify left)
+			)
+		)
+		(property "Value" "120R"
+			(at 59.69 58.4199 0)
+			(effects
+				(font
+					(size 1.27 1.27)
+				)
+				(justify left)
+			)
+		)
+		(property "Footprint" "Resistor_SMD:R_0603_1608Metric_Pad0.98x0.95mm_HandSolder"
+			(at 55.372 57.15 90)
+			(effects
+				(font
+					(size 1.27 1.27)
+				)
+				(hide yes)
+			)
+		)
+		(property "Datasheet" "~"
+			(at 57.15 57.15 0)
+			(effects
+				(font
+					(size 1.27 1.27)
+				)
+				(hide yes)
+			)
+		)
+		(property "Description" "Resistor"
+			(at 57.15 57.15 0)
+			(effects
+				(font
+					(size 1.27 1.27)
+				)
+				(hide yes)
+			)
+		)
+		(pin "1"
+		)
+		(pin "2"
+		)
+		(instances
+			(project ""
+				(path "/3aee14c3-5480-4f7c-989e-3fef81779034/9be8b538-d844-48b8-8166-3cb7d05a381c/4bfedfbb-7ec6-4f71-829f-70c8eaa097f0"
+					(reference "R90")
+					(unit 1)
+				)
+				(path "/3aee14c3-5480-4f7c-989e-3fef81779034/9be8b538-d844-48b8-8166-3cb7d05a381c/e0dbc6bc-1e73-41c8-9910-a38105ce9a35"
+					(reference "R91")
+					(unit 1)
+				)

Commit message: CAN updated
Parts:
- removed D21: SP0503BAHTG, SP0503BAHTG, symbol 0_SamacSys_Parts:SP0503BAHTG
- added IC8: ESD2CAN24DBZRQ1, SOT95P237X112-3N, symbol 0_SamacSys_Parts:ESD2CAN24DBZRQ1
Connections:
- net GND: now also IC8.3 (GND)
- net HI: now also IC8.2 (IO_2)
- net LO: now also IC8.1 (IO_1)
- no-connect marks 2 -> 1

Commit message: updated ethernet
Parts:
- added TP12: CAN_H, TestPoint:TestPoint_THTPad_D2.0mm_Drill1.0mm, symbol Connector:TestPoint
- added TP14: CAN_L, TestPoint:TestPoint_THTPad_D2.0mm_Drill1.0mm, symbol Connector:TestPoint
Connections:
- net HI: now also TP12.1
- net LO: now also TP14.1
Changed lines of the file:
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@@
+	)
+	(junction
+		(at 71.12 53.34)
+		(diameter 0)
+		(color 0 0 0 0)
+	)
+	(junction
+		(at 71.12 60.96)
+		(diameter 0)
+		(color 0 0 0 0)
 	)
 	(junction
@@
 	(wire
 		(pts
+			(xy 71.12 50.8) (xy 71.12 53.34)
+		)
+		(stroke
+			(width 0)
+			(type default)
+		)
+	)
+	(wire
+		(pts
 			(xy 101.6 36.83) (xy 101.6 38.1)
 		)
@@
 	(wire
 		(pts
+			(xy 71.12 60.96) (xy 85.09 60.96)
+		)
+		(stroke
+			(width 0)
+			(type default)
+		)
+	)
+	(wire
+		(pts
 			(xy 111.76 60.96) (xy 111.76 66.04)
 		)
@@
 	(wire
 		(pts
+			(xy 71.12 53.34) (xy 82.55 53.34)
+		)
+		(stroke
+			(width 0)
+			(type default)
+		)
+	)
+	(wire
+		(pts
 			(xy 26.67 26.67) (xy 25.4 26.67)
 		)
@@
 	(wire
 		(pts
-			(xy 57.15 53.34) (xy 82.55 53.34)
+			(xy 57.15 53.34) (xy 71.12 53.34)
 		)
 		(stroke
@@
 	(wire
 		(pts
-			(xy 57.15 60.96) (xy 85.09 60.96)
+			(xy 71.12 60.96) (xy 71.12 63.5)
+		)
+		(stroke
+			(width 0)
+			(type default)
+		)
+	)
+	(wire
+		(pts
+			(xy 57.15 60.96) (xy 71.12 60.96)
 		)
 		(stroke
@@
 			)
 			(justify right)
+		)
+	)
+	(symbol
+		(lib_id "Connector:TestPoint")
+		(at 71.12 63.5 0)
+		(mirror x)
+		(unit 1)
+		(exclude_from_sim no)
+		(in_bom yes)
+		(on_board yes)
+		(dnp no)
+		(property "Reference" "TP14"
+			(at 73.66 68.0721 0)
+			(effects
+				(font
+					(size 1.27 1.27)
+				)
+				(justify left)
+			)
+		)
+		(property "Value" "CAN_L"
+			(at 73.66 65.5321 0)
+			(effects
+				(font
+					(size 1.27 1.27)
+				)
+				(justify left)
+			)
+		)
+		(property "Footprint" "TestPoint:TestPoint_THTPad_D2.0mm_Drill1.0mm"
+			(at 76.2 63.5 0)
+			(effects
+				(font
+					(size 1.27 1.27)
+				)
+				(hide yes)
+			)
+		)
+		(property "Datasheet" "~"
+			(at 76.2 63.5 0)
+			(effects
+				(font
+					(size 1.27 1.27)
+				)
+				(hide yes)
+			)
+		)
+		(property "Description" "test point"
+			(at 71.12 63.5 0)
+			(effects
+				(font
+					(size 1.27 1.27)
+				)
+				(hide yes)
+			)
+		)
+		(pin "1"
+		)
+		(instances
+			(project "NCU"
+				(path "/3aee14c3-5480-4f7c-989e-3fef81779034/9be8b538-d844-48b8-8166-3cb7d05a381c/4bfedfbb-7ec6-4f71-829f-70c8eaa097f0"
+					(reference "TP14")
+					(unit 1)
+				)
+				(path "/3aee14c3-5480-4f7c-989e-3fef81779034/9be8b538-d844-48b8-8166-3cb7d05a381c/e0dbc6bc-1e73-41c8-9910-a38105ce9a35"
+					(reference "TP15")
+					(unit 1)
+				)
+			)
 		)
 	)
@@
 					(unit 1)
 				)
+			)
+		)
+	)
+	(symbol
+		(lib_id "Connector:TestPoint")
+		(at 71.12 50.8 0)
+		(unit 1)
+		(exclude_from_sim no)
+		(in_bom yes)
+		(on_board yes)
+		(dnp no)
+		(fields_autoplaced yes)
+		(property "Reference" "TP12"
+			(at 73.66 46.2279 0)
+			(effects
+				(font
+					(size 1.27 1.27)
+				)
+				(justify left)
+			)
+		)
+		(property "Value" "CAN_H"
+			(at 73.66 48.7679 0)
+			(effects
+				(font
+					(size 1.27 1.27)
+				)
+				(justify left)
+			)
+		)
+		(property "Footprint" "TestPoint:TestPoint_THTPad_D2.0mm_Drill1.0mm"
+			(at 76.2 50.8 0)
+			(effects
+				(font
+					(size 1.27 1.27)
+				)
+				(hide yes)
+			)
+		)
+		(property "Datasheet" "~"
+			(at 76.2 50.8 0)
+			(effects
+				(font
+					(size 1.27 1.27)
+				)
+				(hide yes)
+			)
+		)
+		(property "Description" "test point"
+			(at 71.12 50.8 0)
+			(effects
+				(font
+					(size 1.27 1.27)
+				)
+				(hide yes)
+			)
+		)
+		(pin "1"
+		)
+		(instances
+			(project "NCU"
+				(path "/3aee14c3-5480-4f7c-989e-3fef81779034/9be8b538-d844-48b8-8166-3cb7d05a381c/4bfedfbb-7ec6-4f71-829f-70c8eaa097f0"
+					(reference "TP12")
+					(unit 1)
+				)
+				(path "/3aee14c3-5480-4f7c-989e-3fef81779034/9be8b538-d844-48b8-8166-3cb7d05a381c/e0dbc6bc-1e73-41c8-9910-a38105ce9a35"
+					(reference "TP13")
+					(unit 1)
+				)

Commit message: reannotated, updated some symbols
Parts:
- renumbered C59 to C66, C60 to C67, IC8 to IC3, R90 to R85, TP12 to TP14, TP14 to TP15, U2 to U4
Changed lines of the file:
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@@
 		(on_board yes)
 		(dnp no)
-		(property "Reference" "TP14"
+		(property "Reference" "TP15"
 			(at 73.66 68.0721 0)
 			(effects
@@
 			(project "NCU"
 				(path "/3aee14c3-5480-4f7c-989e-3fef81779034/9be8b538-d844-48b8-8166-3cb7d05a381c/4bfedfbb-7ec6-4f71-829f-70c8eaa097f0"
-					(reference "TP14")
-					(unit 1)
-				)
-				(path "/3aee14c3-5480-4f7c-989e-3fef81779034/9be8b538-d844-48b8-8166-3cb7d05a381c/e0dbc6bc-1e73-41c8-9910-a38105ce9a35"
 					(reference "TP15")
+					(unit 1)
+				)
+				(path "/3aee14c3-5480-4f7c-989e-3fef81779034/9be8b538-d844-48b8-8166-3cb7d05a381c/e0dbc6bc-1e73-41c8-9910-a38105ce9a35"
+					(reference "TP17")
 					(unit 1)
 				)
@@
 		(on_board yes)
 		(dnp no)
-		(property "Reference" "#PWR0236"
+		(property "Reference" "#PWR0317"
 			(at 26.67 29.21 0)
 			(effects
@@
 			(project "NCU"
 				(path "/3aee14c3-5480-4f7c-989e-3fef81779034/9be8b538-d844-48b8-8166-3cb7d05a381c/4bfedfbb-7ec6-4f71-829f-70c8eaa097f0"
-					(reference "#PWR0236")
-					(unit 1)
-				)
-				(path "/3aee14c3-5480-4f7c-989e-3fef81779034/9be8b538-d844-48b8-8166-3cb7d05a381c/e0dbc6bc-1e73-41c8-9910-a38105ce9a35"
-					(reference "#PWR0258")
+					(reference "#PWR0317")
+					(unit 1)
+				)
+				(path "/3aee14c3-5480-4f7c-989e-3fef81779034/9be8b538-d844-48b8-8166-3cb7d05a381c/e0dbc6bc-1e73-41c8-9910-a38105ce9a35"
+					(reference "#PWR0352")
 					(unit 1)
 				)
@@
 		(dnp no)
 		(fields_autoplaced yes)
-		(property "Reference" "C59"
+		(property "Reference" "C66"
 			(at 111.76 40.6399 0)
 			(effects
@@
 			(project "NCU"
 				(path "/3aee14c3-5480-4f7c-989e-3fef81779034/9be8b538-d844-48b8-8166-3cb7d05a381c/4bfedfbb-7ec6-4f71-829f-70c8eaa097f0"
-					(reference "C59")
-					(unit 1)
-				)
-				(path "/3aee14c3-5480-4f7c-989e-3fef81779034/9be8b538-d844-48b8-8166-3cb7d05a381c/e0dbc6bc-1e73-41c8-9910-a38105ce9a35"
-					(reference "C64")
+					(reference "C66")
+					(unit 1)
+				)
+				(path "/3aee14c3-5480-4f7c-989e-3fef81779034/9be8b538-d844-48b8-8166-3cb7d05a381c/e0dbc6bc-1e73-41c8-9910-a38105ce9a35"
+					(reference "C71")
 					(unit 1)
 				)
@@
 		(on_board yes)
 		(dnp no)
-		(property "Reference" "#PWR0241"
+		(property "Reference" "#PWR0322"
 			(at 118.11 93.98 0)
 			(effects
@@
 			(project "NCU"
 				(path "/3aee14c3-5480-4f7c-989e-3fef81779034/9be8b538-d844-48b8-8166-3cb7d05a381c/4bfedfbb-7ec6-4f71-829f-70c8eaa097f0"
-					(reference "#PWR0241")
-					(unit 1)
-				)
-				(path "/3aee14c3-5480-4f7c-989e-3fef81779034/9be8b538-d844-48b8-8166-3cb7d05a381c/e0dbc6bc-1e73-41c8-9910-a38105ce9a35"
-					(reference "#PWR0263")
+					(reference "#PWR0322")
+					(unit 1)
+				)
+				(path "/3aee14c3-5480-4f7c-989e-3fef81779034/9be8b538-d844-48b8-8166-3cb7d05a381c/e0dbc6bc-1e73-41c8-9910-a38105ce9a35"
+					(reference "#PWR0357")
 					(unit 1)
 				)
@@
 		(on_board yes)
 		(dnp no)
-		(property "Reference" "#PWR0239"
+		(property "Reference" "#PWR0320"
 			(at 101.6 72.39 0)
 			(effects
@@
 			(project "NCU"
 				(path "/3aee14c3-5480-4f7c-989e-3fef81779034/9be8b538-d844-48b8-8166-3cb7d05a381c/4bfedfbb-7ec6-4f71-829f-70c8eaa097f0"
-					(reference "#PWR0239")
-					(unit 1)
-				)
-				(path "/3aee14c3-5480-4f7c-989e-3fef81779034/9be8b538-d844-48b8-8166-3cb7d05a381c/e0dbc6bc-1e73-41c8-9910-a38105ce9a35"
-					(reference "#PWR0261")
+					(reference "#PWR0320")
+					(unit 1)
+				)
+				(path "/3aee14c3-5480-4f7c-989e-3fef81779034/9be8b538-d844-48b8-8166-3cb7d05a381c/e0dbc6bc-1e73-41c8-9910-a38105ce9a35"
+					(reference "#PWR0355")
 					(unit 1)
 				)
@@
 		(dnp no)
 		(fields_autoplaced yes)
-		(property "Reference" "IC8"
+		(property "Reference" "IC3"
 			(at 101.6 76.2 0)
 			(effects
@@
 			(project ""
 				(path "/3aee14c3-5480-4f7c-989e-3fef81779034/9be8b538-d844-48b8-8166-3cb7d05a381c/4bfedfbb-7ec6-4f71-829f-70c8eaa097f0"
-					(reference "IC8")
-					(unit 1)
-				)
-				(path "/3aee14c3-5480-4f7c-989e-3fef81779034/9be8b538-d844-48b8-8166-3cb7d05a381c/e0dbc6bc-1e73-41c8-9910-a38105ce9a35"
-					(reference "IC9")
+					(reference "IC3")
+					(unit 1)
+				)
+				(path "/3aee14c3-5480-4f7c-989e-3fef81779034/9be8b538-d844-48b8-8166-3cb7d05a381c/e0dbc6bc-1e73-41c8-9910-a38105ce9a35"
+					(reference "IC5")
 					(unit 1)
 				)
@@
 		(on_board yes)
 		(dnp no)
-		(property "Reference" "U2"
+		(property "Reference" "U4"
 			(at 99.4567 45.72 0)
 			(effects
@@
 			(project "NCU"
 				(path "/3aee14c3-5480-4f7c-989e-3fef81779034/9be8b538-d844-48b8-8166-3cb7d05a381c/4bfedfbb-7ec6-4f71-829f-70c8eaa097f0"
-					(reference "U2")
-					(unit 1)
-				)
-				(path "/3aee14c3-5480-4f7c-989e-3fef81779034/9be8b538-d844-48b8-8166-3cb7d05a381c/e0dbc6bc-1e73-41c8-9910-a38105ce9a35"
-					(reference "U3")
+					(reference "U4")
+					(unit 1)
+				)
+				(path "/3aee14c3-5480-4f7c-989e-3fef81779034/9be8b538-d844-48b8-8166-3cb7d05a381c/e0dbc6bc-1e73-41c8-9910-a38105ce9a35"
+					(reference "U5")
 					(unit 1)
 				)
@@
 		(dnp no)
 		(fields_autoplaced yes)
-		(property "Reference" "TP12"
+		(property "Reference" "TP14"
 			(at 73.66 46.2279 0)
 			(effects
@@
 			(project "NCU"
 				(path "/3aee14c3-5480-4f7c-989e-3fef81779034/9be8b538-d844-48b8-8166-3cb7d05a381c/4bfedfbb-7ec6-4f71-829f-70c8eaa097f0"
-					(reference "TP12")
-					(unit 1)
-				)
-				(path "/3aee14c3-5480-4f7c-989e-3fef81779034/9be8b538-d844-48b8-8166-3cb7d05a381c/e0dbc6bc-1e73-41c8-9910-a38105ce9a35"
-					(reference "TP13")
+					(reference "TP14")
+					(unit 1)
+				)
+				(path "/3aee14c3-5480-4f7c-989e-3fef81779034/9be8b538-d844-48b8-8166-3cb7d05a381c/e0dbc6bc-1e73-41c8-9910-a38105ce9a35"
+					(reference "TP16")
 					(unit 1)
 				)
@@
 		(on_board yes)
 		(dnp no)
-		(property "Reference" "#PWR0237"
+		(property "Reference" "#PWR0318"
 			(at 26.67 36.83 0)
 			(effects
@@
 			(project "NCU"
 				(path "/3aee14c3-5480-4f7c-989e-3fef81779034/9be8b538-d844-48b8-8166-3cb7d05a381c/4bfedfbb-7ec6-4f71-829f-70c8eaa097f0"
-					(reference "#PWR0237")
-					(unit 1)
-				)
-				(path "/3aee14c3-5480-4f7c-989e-3fef81779034/9be8b538-d844-48b8-8166-3cb7d05a381c/e0dbc6bc-1e73-41c8-9910-a38105ce9a35"
-					(reference "#PWR0259")
+					(reference "#PWR0318")
+					(unit 1)
+				)
+				(path "/3aee14c3-5480-4f7c-989e-3fef81779034/9be8b538-d844-48b8-8166-3cb7d05a381c/e0dbc6bc-1e73-41c8-9910-a38105ce9a35"
+					(reference "#PWR0353")
 					(unit 1)
 				)
@@
 		(dnp no)
 		(fields_autoplaced yes)
-		(property "Reference" "#PWR0240"
+		(property "Reference" "#PWR0321"
 			(at 118.11 52.07 0)
 			(effects
@@
 			(project "NCU"
 				(path "/3aee14c3-5480-4f7c-989e-3fef81779034/9be8b538-d844-48b8-8166-3cb7d05a381c/4bfedfbb-7ec6-4f71-829f-70c8eaa097f0"
-					(reference "#PWR0240")
-					(unit 1)
-				)
-				(path "/3aee14c3-5480-4f7c-989e-3fef81779034/9be8b538-d844-48b8-8166-3cb7d05a381c/e0dbc6bc-1e73-41c8-9910-a38105ce9a35"
-					(reference "#PWR0262")
+					(reference "#PWR0321")
+					(unit 1)
+				)
+				(path "/3aee14c3-5480-4f7c-989e-3fef81779034/9be8b538-d844-48b8-8166-3cb7d05a381c/e0dbc6bc-1e73-41c8-9910-a38105ce9a35"
+					(reference "#PWR0356")
 					(unit 1)
 				)
@@
 		(dnp yes)
 		(fields_autoplaced yes)
-		(property "Reference" "R90"
+		(property "Reference" "R85"
 			(at 59.69 55.8799 0)
 			(effects
@@
 			(project ""
 				(path "/3aee14c3-5480-4f7c-989e-3fef81779034/9be8b538-d844-48b8-8166-3cb7d05a381c/4bfedfbb-7ec6-4f71-829f-70c8eaa097f0"
-					(reference "R90")
-					(unit 1)
-				)
-				(path "/3aee14c3-5480-4f7c-989e-3fef81779034/9be8b538-d844-48b8-8166-3cb7d05a381c/e0dbc6bc-1e73-41c8-9910-a38105ce9a35"
-					(reference "R91")
+					(reference "R85")
+					(unit 1)
+				)
+				(path "/3aee14c3-5480-4f7c-989e-3fef81779034/9be8b538-d844-48b8-8166-3cb7d05a381c/e0dbc6bc-1e73-41c8-9910-a38105ce9a35"
+					(reference "R109")
 					(unit 1)
 				)
@@
 		(on_board yes)
 		(dnp no)
-		(property "Reference" "#PWR0238"
+		(property "Reference" "#PWR0319"
 			(at 101.6 40.64 0)
 			(effects
@@
 			(project "NCU"
 				(path "/3aee14c3-5480-4f7c-989e-3fef81779034/9be8b538-d844-48b8-8166-3cb7d05a381c/4bfedfbb-7ec6-4f71-829f-70c8eaa097f0"
-					(reference "#PWR0238")
-					(unit 1)
-				)
-				(path "/3aee14c3-5480-4f7c-989e-3fef81779034/9be8b538-d844-48b8-8166-3cb7d05a381c/e0dbc6bc-1e73-41c8-9910-a38105ce9a35"
-					(reference "#PWR0260")
+					(reference "#PWR0319")
+					(unit 1)
+				)
+				(path "/3aee14c3-5480-4f7c-989e-3fef81779034/9be8b538-d844-48b8-8166-3cb7d05a381c/e0dbc6bc-1e73-41c8-9910-a38105ce9a35"
+					(reference "#PWR0354")
 					(unit 1)
 				)
@@
 		(dnp no)
 		(fields_autoplaced yes)
-		(property "Reference" "C60"
+		(property "Reference" "C67"
 			(at 121.92 40.6399 0)
 			(effects
@@
 			(project "NCU"
 				(path "/3aee14c3-5480-4f7c-989e-3fef81779034/9be8b538-d844-48b8-8166-3cb7d05a381c/4bfedfbb-7ec6-4f71-829f-70c8eaa097f0"
-					(reference "C60")
-					(unit 1)
-				)
-				(path "/3aee14c3-5480-4f7c-989e-3fef81779034/9be8b538-d844-48b8-8166-3cb7d05a381c/e0dbc6bc-1e73-41c8-9910-a38105ce9a35"
-					(reference "C65")
-					(unit 1)
-				)
+					(reference "C67")
+					(unit 1)
+				)
+				(path "/3aee14c3-5480-4f7c-989e-3fef81779034/9be8b538-d844-48b8-8166-3cb7d05a381c/e0dbc6bc-1e73-41c8-9910-a38105ce9a35"
+					(reference "C72")
+					(unit 1)
+				)

Commit message: updates from bom release
Parts:
- R85: value 120R -> 120
Changed lines of the file:
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@@
 			)
 		)
-		(property "Value" "120R"
+		(property "Value" "120"
 			(at 59.69 58.4199 0)
 			(effects
