File: pcb/HSD.kicad_sch (KiCad schematic)
At the start: 11 parts, among them IC1 VND7E025AJTR

Commit message: added USB protection, reviewed LSD and HSD, improved input TVS footprint
Parts:
- removed D8: BAT54W, Package_TO_SOT_SMD:SOT-323_SC-70, symbol Diode:BAT54W
- added D7: 1N4148, Diode_THT:D_DO-35_SOD27_P7.62mm_Horizontal, symbol Diode:1N4148
- added R1: 15k, Resistor_SMD:R_0603_1608Metric_Pad0.98x0.95mm_HandSolder, symbol Device:R
- added R100, R3: 100k, Resistor_SMD:R_0603_1608Metric_Pad0.98x0.95mm_HandSolder, symbol Device:R
Connections:
- net CTRL_A: now also R3.1
- net CTRL_B: now also R100.1
- net GND: now also D7.1 (K), R100.2, R3.2
- net ISEN: now also R1.1; no longer IC1.7 (CS), R24.2
- net at IC1.4 (GND), R25.1: now also D7.2 (A)
- new net: IC1.7 (CS), R1.2, R24.2
Other:
- moved on the sheet: C37, C38, IC1, R20, R21, R22, R23, R24, R25, R26

Commit message: reannotated, updated some symbols
Parts:
- renumbered C37 to C42, C38 to C43, R3 to R24, R100 to R25, R20 to R26, R21 to R27, R22 to R28, R1 to R29, R23 to R30, R24 to R31, R25 to R32, R26 to R33

Commit message: initial hsd layout
Parts:
- D7: value 1N4148 -> 1N4148W; footprint Diode_THT:D_DO-35_SOD27_P7.62mm_Horizontal -> Diode_SMD:D_SOD-123; symbol Diode:1N4148 -> Diode:1N4148W
Changed lines of the file:
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@@
 	)
 	(symbol
-		(lib_id "Diode:1N4148")
+		(lib_id "Diode:1N4148W")
 		(at 111.76 63.5 90)
 		(unit 1)
@@
 			)
 		)
-		(property "Value" "1N4148"
+		(property "Value" "1N4148W"
 			(at 114.3 64.7699 90)
 			(effects
@@
 			)
 		)
-		(property "Footprint" "Diode_THT:D_DO-35_SOD27_P7.62mm_Horizontal"
+		(property "Footprint" "Diode_SMD:D_SOD-123"
+			(at 116.205 63.5 0)
+			(effects
+				(font
+					(size 1.27 1.27)
+				)
+				(hide yes)
+			)
+		)
+		(property "Datasheet" "https://www.vishay.com/docs/85748/1n4148w.pdf"
 			(at 111.76 63.5 0)
 			(effects
@@
 			)
 		)
-		(property "Datasheet" "https://assets.nexperia.com/documents/data-sheet/1N4148_1N4448.pdf"
+		(property "Description" "75V 0.15A Fast Switching Diode, SOD-123"
 			(at 111.76 63.5 0)
 			(effects
-				(font
-					(size 1.27 1.27)
-				)
-				(hide yes)
-			)
-		)
-		(property "Description" "100V 0.15A standard switching diode, DO-35"
-			(at 111.76 63.5 0)
-			(effects

Commit message: updates from bom release
Parts:
- R31: value 620R -> 620
Changed lines of the file:
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@@
 			)
 		)
-		(property "Value" "620R"
+		(property "Value" "620"
 			(at 98.298 64.77 0)
 			(effects
