File: pcb/INPUT_20V.kicad_sch (KiCad schematic)
At the start: 5 parts

Commit message: updated ethernet
Parts:
- removed C46: 100nF, Capacitor_SMD:C_0603_1608Metric_Pad1.08x0.95mm_HandSolder, symbol Device:C
- removed D14: BZV55C3V6, Diode_SMD:D_MiniMELF, symbol Diode:BZV55C3V6
- removed R41: 100, Resistor_SMD:R_0603_1608Metric_Pad0.98x0.95mm_HandSolder, symbol Device:R
- removed R42: 10k, Resistor_SMD:R_0603_1608Metric_Pad0.98x0.95mm_HandSolder, symbol Device:R
- removed R43: 1k, Resistor_SMD:R_0603_1608Metric_Pad0.98x0.95mm_HandSolder, symbol Device:R
- added C87: 100nF, Capacitor_SMD:C_0603_1608Metric_Pad1.08x0.95mm_HandSolder, symbol Device:C
- added D5: BAT54S, Package_TO_SOT_SMD:SOT-23, symbol Diode:BAT54S
- added R13: 8.2k, Resistor_SMD:R_0603_1608Metric_Pad0.98x0.95mm_HandSolder, symbol Device:R
- added R30: 1k, Resistor_SMD:R_0603_1608Metric_Pad0.98x0.95mm_HandSolder, symbol Device:R
- added R38: 100, Resistor_SMD:R_0603_1608Metric_Pad0.98x0.95mm_HandSolder, symbol Device:R
Connections:
- new net: R13.2, R30.1, R38.1
- new net 3V3: D5.2 (K)
- new net AGND: C87.2, D5.1 (A), R30.2
- new net INPUT: R13.1
- new net OUTPUT: C87.1, D5.3, R38.2

Commit message: reannotated, updated some symbols
Parts:
- renumbered C87 to C52, D5 to D16, R13 to R53, R30 to R54, R38 to R55

Commit message: removed AGND and added ground garden
Connections:
- net AGND is gone; now on net GND: C52.2, D16.1 (A), R54.2
Changed lines of the file:
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@@
 			)
 		)
-		(property "Value" "AGND"
+		(property "Value" "GND"
 			(at 88.9 73.66 0)
 			(effects
@@
 			)
 		)
-		(property "Value" "AGND"
+		(property "Value" "GND"
 			(at 114.3 73.66 0)
 			(effects
@@
 			)
 		)
-		(property "Value" "AGND"
+		(property "Value" "GND"
 			(at 133.35 73.66 0)
 			(effects

Commit message: updates from bom release
Parts:
- C52: value 100nF -> 100n
Changed lines of the file:
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@@
 			)
 		)
-		(property "Value" "100nF"
+		(property "Value" "100n"
 			(at 117.348 64.77 0)
 			(effects
