File: pcb/MCUPower.kicad_sch (KiCad schematic)
At the start: 31 parts

Commit message: reannotated, updated some symbols
Parts:
- added JP6, JP7, JP8: SolderJumper_2_Bridged, Jumper:SolderJumper-2_P1.3mm_Bridged_RoundedPad1.0x1.5mm, symbol Jumper:SolderJumper_2_Bridged
- renumbered C8 to C13, C9 to C14, C10 to C15, C11 to C16, C12 to C17, C13 to C18, C14 to C19, C15 to C20, C16 to C21, C17 to C22, C18 to C23, C19 to C24, C20 to C25, C21 to C26, C22 to C27, C23 to C28, C24 to C29, C25 to C30, C26 to C31, C27 to C32, C28 to C33, C29 to C34, C30 to C35, C31 to C36, C32 to C37, C33 to C38, C34 to C39, C35 to C40, C36 to C41, FB1 to FB2
Connections:
- net VCAP: now also JP6.1 (A)
- net VDDA: now also JP8.2 (B); no longer C39.1, C41.1
- net VDDLDO: now also JP7.1 (A); no longer C34.1, L1.2
- new net 1V2_MCU: C34.1, JP7.2 (B), L1.2
- new net VFBSMPS: JP6.2 (B)
- new net VREF+: C39.1, C41.1, JP8.1 (A)

Commit message: initial microcontroller layout
Parts:
- removed L1: VLS3015CX-2R2M-H, VLS3015, symbol 0_SamacSys_Parts:VLS3015CX-2R2M-H
- added L1: 2.2uH, Inductor_SMD:L_0805_2012Metric_Pad1.05x1.20mm_HandSolder, symbol Device:L
Connections:
- net 1V2_MCU: now also L1.2
- net VLXSMPS: now also L1.1
Changed lines of the file:
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@@
 		)
 	)
+	(text_box "This should be a copper pour possibly under the STM on the power layer"
+		(exclude_from_sim no)
+		(at 232.41 66.04 0)
+		(size 24.13 3.81)
+		(margins 0.9525 0.9525 0.9525 0.9525)
+		(stroke
+			(width -0.0001)
+			(type solid)
+		)
+		(fill
+			(type none)
+		)
+		(effects
+			(font
+				(size 1.016 1.016)
+			)
+			(justify left top)
+		)
+	)
 	(junction
 		(at 139.7 38.1)
@@
 	)
 	(junction
-		(at 31.75 38.1)
+		(at 228.6 76.2)
 		(diameter 0)
 		(color 0 0 0 0)
 	)
 	(junction
-		(at 76.2 76.2)
+		(at 31.75 38.1)
 		(diameter 0)
 		(color 0 0 0 0)
 	)
 	(junction
-		(at 50.8 38.1)
+		(at 76.2 76.2)
 		(diameter 0)
 		(color 0 0 0 0)
 	)
 	(junction
-		(at 208.28 76.2)
+		(at 50.8 38.1)
 		(diameter 0)
 		(color 0 0 0 0)
@@
 	)
 	(junction
+		(at 208.28 76.2)
+		(diameter 0)
+		(color 0 0 0 0)
+	)
+	(junction
 		(at 224.79 113.03)
 		(diameter 0)
@@
 	)
 	(junction
-		(at 228.6 76.2)
-		(diameter 0)
-		(color 0 0 0 0)
-	)
-	(junction
 		(at 152.4 38.1)
 		(diameter 0)
@@
 	(wire
 		(pts
+			(xy 208.28 76.2) (xy 214.63 76.2)
+		)
+		(stroke
+			(width 0)
+			(type default)
+		)
+	)
+	(wire
+		(pts
 			(xy 101.6 38.1) (xy 114.3 38.1)
 		)
@@
 		)
 	)
+	(wire
+		(pts
+			(xy 222.25 76.2) (xy 228.6 76.2)
+		)
+		(stroke
+			(width 0)
+			(type default)
+		)
+	)
 	(label "1V2_MCU"
 		(at 234.95 76.2 0)
@@
 	)
 	(symbol
+		(lib_id "Device:L")
+		(at 218.44 76.2 90)
+		(unit 1)
+		(exclude_from_sim no)
+		(in_bom yes)
+		(on_board yes)
+		(dnp no)
+		(fields_autoplaced yes)
+		(property "Reference" "L1"
+			(at 218.44 71.12 90)
+			(effects
+				(font
+					(size 1.27 1.27)
+				)
+			)
+		)
+		(property "Value" "2.2uH"
+			(at 218.44 73.66 90)
+			(effects
+				(font
+					(size 1.27 1.27)
+				)
+			)
+		)
+		(property "Footprint" "Inductor_SMD:L_0805_2012Metric_Pad1.05x1.20mm_HandSolder"
+			(at 218.44 76.2 0)
+			(effects
+				(font
+					(size 1.27 1.27)
+				)
+				(hide yes)
+			)
+		)
+		(property "Datasheet" "DFE201210U-2R2M=P2"
+			(at 218.44 76.2 0)
+			(effects
+				(font
+					(size 1.27 1.27)
+				)
+				(hide yes)
+			)
+		)
+		(property "Description" "Inductor"
+			(at 218.44 76.2 0)
+			(effects
+				(font
+					(size 1.27 1.27)
+				)
+				(hide yes)
+			)
+		)
+		(pin "1"
+		)
+		(pin "2"
+		)
+		(instances
+			(project ""
+				(path "/3aee14c3-5480-4f7c-989e-3fef81779034/d2b1e1a0-8b64-49ff-b975-b40fa2d33dc6/70b8fb88-9c19-46a8-95e3-6c05e68e24c9"
+					(reference "L1")
+					(unit 1)
+				)
+			)
+		)
+	)
+	(symbol
 		(lib_id "Device:C")
 		(at 177.8 44.45 0)
@@
 					(unit 1)
 				)
-			)
-		)
-	)
-	(symbol
-		(lib_id "0_SamacSys_Parts:VLS3015CX-2R2M-H")
-		(at 208.28 76.2 0)
-		(mirror x)
-		(unit 1)
-		(exclude_from_sim no)
-		(in_bom yes)
-		(on_board yes)
-		(dnp no)
-		(fields_autoplaced yes)
-		(property "Reference" "L1"
-			(at 218.44 69.85 0)
-			(effects
-				(font
-					(size 1.27 1.27)
-				)
-			)
-		)
-		(property "Value" "VLS3015CX-2R2M-H"
-			(at 218.44 72.39 0)
-			(effects
-				(font
-					(size 1.27 1.27)
-				)
-			)
-		)
-		(property "Footprint" "VLS3015"
-			(at 224.79 77.47 0)
-			(effects
-				(font
-					(size 1.27 1.27)
-				)
-				(justify left)
-				(hide yes)
-			)
-		)
-		(property "Datasheet" "https://product.tdk.com/system/files/dam/doc/product/inductor/inductor/smd/catalog/inductor_automotive_power_vls3015cx-h_en.pdf"
-			(at 224.79 74.93 0)
-			(effects
-				(font
-					(size 1.27 1.27)
-				)
-				(justify left)
-				(hide yes)
-			)
-		)
-		(property "Description" "SMD / SMT Inductors (Coils), L=2.2?H, L x W x T :"
-			(at 208.28 76.2 0)
-			(effects
-				(font
-					(size 1.27 1.27)
-				)
-				(hide yes)
-			)
-		)
-		(property "Description_1" "SMD / SMT Inductors (Coils), L=2.2?H, L x W x T :"
-			(at 224.79 72.39 0)
-			(effects
-				(font
-					(size 1.27 1.27)
-				)
-				(justify left)
-				(hide yes)
-			)
-		)
-		(property "Height" ""
-			(at 224.79 69.85 0)
-			(effects
-				(font
-					(size 1.27 1.27)
-				)
-				(justify left)
-				(hide yes)
-			)
-		)
-		(property "Mouser Part Number" "810-VLS3015CX-2R2M-H"
-			(at 224.79 67.31 0)
-			(effects
-				(font
-					(size 1.27 1.27)
-				)
-				(justify left)
-				(hide yes)
-			)
-		)
-		(property "Mouser Price/Stock" "https://www.mouser.co.uk/ProductDetail/TDK/VLS3015CX-2R2M-H?qs=zW32dvEIR3uMKTZetq6xLg%3D%3D"
-			(at 224.79 64.77 0)
-			(effects
-				(font
-					(size 1.27 1.27)
-				)
-				(justify left)
-				(hide yes)
-			)
-		)
-		(property "Manufacturer_Name" "TDK"
-			(at 224.79 62.23 0)
-			(effects
-				(font
-					(size 1.27 1.27)
-				)
-				(justify left)
-				(hide yes)
-			)
-		)
-		(property "Manufacturer_Part_Number" "VLS3015CX-2R2M-H"
-			(at 224.79 59.69 0)
-			(effects
-				(font
-					(size 1.27 1.27)
-				)
-				(justify left)
-				(hide yes)
-			)
-		)
-		(pin "1"
-		)
-		(pin "2"
-		)
-		(instances
-			(project "NCU"
-				(path "/3aee14c3-5480-4f7c-989e-3fef81779034/d2b1e1a0-8b64-49ff-b975-b40fa2d33dc6/70b8fb88-9c19-46a8-95e3-6c05e68e24c9"
-					(reference "L1")
-					(unit 1)
-				)

Commit message: routed LSDs to micro
Parts:
- removed JP8: SolderJumper_2_Bridged, Jumper:SolderJumper-2_P1.3mm_Bridged_RoundedPad1.0x1.5mm, symbol Jumper:SolderJumper_2_Bridged
Connections:
- net VREF+ is gone; now on net VDDA: C39.1, C41.1
Changed lines of the file:
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@@
 	(wire
 		(pts
-			(xy 241.3 38.1) (xy 247.65 38.1)
+			(xy 241.3 38.1) (xy 260.35 38.1)
 		)
 		(stroke
@@
 		(pts
 			(xy 88.9 38.1) (xy 88.9 40.64)
-		)
-		(stroke
-			(width 0)
-			(type default)
-		)
-	)
-	(wire
-		(pts
-			(xy 255.27 38.1) (xy 260.35 38.1)
 		)
 		(stroke
@@
 					(unit 1)
 				)
-			)
-		)
-	)
-	(symbol
-		(lib_id "Jumper:SolderJumper_2_Bridged")
-		(at 251.46 38.1 180)
-		(unit 1)
-		(exclude_from_sim no)
-		(in_bom no)
-		(on_board yes)
-		(dnp no)
-		(property "Reference" "JP8"
-			(at 249.936 35.56 0)
-			(effects
-				(font
-					(size 1.27 1.27)
-				)
-				(justify right)
-			)
-		)
-		(property "Value" "SolderJumper_2_Bridged"
-			(at 252.7299 35.56 90)
-			(effects
-				(font
-					(size 1.27 1.27)
-				)
-				(justify right)
-				(hide yes)
-			)
-		)
-		(property "Footprint" "Jumper:SolderJumper-2_P1.3mm_Bridged_RoundedPad1.0x1.5mm"
-			(at 251.46 38.1 0)
-			(effects
-				(font
-					(size 1.27 1.27)
-				)
-				(hide yes)
-			)
-		)
-		(property "Datasheet" "~"
-			(at 251.46 38.1 0)
-			(effects
-				(font
-					(size 1.27 1.27)
-				)
-				(hide yes)
-			)
-		)
-		(property "Description" "Solder Jumper, 2-pole, closed/bridged"
-			(at 251.46 38.1 0)
-			(effects
-				(font
-					(size 1.27 1.27)
-				)
-				(hide yes)
-			)
-		)
-		(pin "2"
-		)
-		(pin "1"
-		)
-		(instances
-			(project "NCU"
-				(path "/3aee14c3-5480-4f7c-989e-3fef81779034/d2b1e1a0-8b64-49ff-b975-b40fa2d33dc6/70b8fb88-9c19-46a8-95e3-6c05e68e24c9"
-					(reference "JP8")
-					(unit 1)
-				)

Commit message: removed solder jumpers for mcu power scheme, as taking up too much space on the board
Parts:
- removed JP6, JP7: SolderJumper_2_Bridged, Jumper:SolderJumper-2_P1.3mm_Bridged_RoundedPad1.0x1.5mm, symbol Jumper:SolderJumper_2_Bridged
Connections:
- net 1V2_MCU is gone; now on net VDDLDO: C34.1, L1.2
Changed lines of the file:
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@@
 	(wire
 		(pts
-			(xy 252.73 76.2) (xy 254 76.2)
-		)
-		(stroke
-			(width 0)
-			(type default)
-		)
-	)
-	(wire
-		(pts
 			(xy 152.4 35.56) (xy 152.4 38.1)
 		)
@@
 	(wire
 		(pts
-			(xy 224.79 99.06) (xy 224.79 102.87)
+			(xy 224.79 99.06) (xy 224.79 113.03)
 		)
 		(stroke
@@
 	(wire
 		(pts
-			(xy 228.6 76.2) (xy 245.11 76.2)
+			(xy 228.6 76.2) (xy 254 76.2)
 		)
 		(stroke
@@
 	(wire
 		(pts
-			(xy 224.79 110.49) (xy 224.79 113.03)
-		)
-		(stroke
-			(width 0)
-			(type default)
-		)
-	)
-	(wire
-		(pts
 			(xy 254 86.36) (xy 254 88.9)
 		)
@@
 		)
 	)
-	(label "1V2_MCU"
-		(at 234.95 76.2 0)
-		(effects
-			(font
-				(size 1.27 1.27)
-			)
-			(justify left bottom)
-		)
-	)
 	(hierarchical_label "VDD"
 		(shape passive)
@@
 	)
 	(symbol
-		(lib_id "Jumper:SolderJumper_2_Bridged")
-		(at 224.79 106.68 90)
-		(unit 1)
-		(exclude_from_sim no)
-		(in_bom no)
-		(on_board yes)
-		(dnp no)
-		(property "Reference" "JP6"
-			(at 226.314 106.68 90)
-			(effects
-				(font
-					(size 1.27 1.27)
-				)
-				(justify right)
-			)
-		)
-		(property "Value" "SolderJumper_2_Bridged"
-			(at 227.33 107.9499 90)
-			(effects
-				(font
-					(size 1.27 1.27)
-				)
-				(justify right)
-				(hide yes)
-			)
-		)
-		(property "Footprint" "Jumper:SolderJumper-2_P1.3mm_Bridged_RoundedPad1.0x1.5mm"
-			(at 224.79 106.68 0)
-			(effects
-				(font
-					(size 1.27 1.27)
-				)
-				(hide yes)
-			)
-		)
-		(property "Datasheet" "~"
-			(at 224.79 106.68 0)
-			(effects
-				(font
-					(size 1.27 1.27)
-				)
-				(hide yes)
-			)
-		)
-		(property "Description" "Solder Jumper, 2-pole, closed/bridged"
-			(at 224.79 106.68 0)
-			(effects
-				(font
-					(size 1.27 1.27)
-				)
-				(hide yes)
-			)
-		)
-		(pin "2"
-		)
-		(pin "1"
-		)
-		(instances
-			(project ""
-				(path "/3aee14c3-5480-4f7c-989e-3fef81779034/d2b1e1a0-8b64-49ff-b975-b40fa2d33dc6/70b8fb88-9c19-46a8-95e3-6c05e68e24c9"
-					(reference "JP6")
-					(unit 1)
-				)
-			)
-		)
-	)
-	(symbol
 		(lib_id "Device:C")
 		(at 228.6 44.45 0)
@@
 					(unit 1)
 				)
-			)
-		)
-	)
-	(symbol
-		(lib_id "Jumper:SolderJumper_2_Bridged")
-		(at 248.92 76.2 180)
-		(unit 1)
-		(exclude_from_sim no)
-		(in_bom no)
-		(on_board yes)
-		(dnp no)
-		(property "Reference" "JP7"
-			(at 247.396 73.66 0)
-			(effects
-				(font
-					(size 1.27 1.27)
-				)
-				(justify right)
-			)
-		)
-		(property "Value" "SolderJumper_2_Bridged"
-			(at 250.1899 73.66 90)
-			(effects
-				(font
-					(size 1.27 1.27)
-				)
-				(justify right)
-				(hide yes)
-			)
-		)
-		(property "Footprint" "Jumper:SolderJumper-2_P1.3mm_Bridged_RoundedPad1.0x1.5mm"
-			(at 248.92 76.2 0)
-			(effects
-				(font
-					(size 1.27 1.27)
-				)
-				(hide yes)
-			)
-		)
-		(property "Datasheet" "~"
-			(at 248.92 76.2 0)
-			(effects
-				(font
-					(size 1.27 1.27)
-				)
-				(hide yes)
-			)
-		)
-		(property "Description" "Solder Jumper, 2-pole, closed/bridged"
-			(at 248.92 76.2 0)
-			(effects
-				(font
-					(size 1.27 1.27)
-				)
-				(hide yes)
-			)
-		)
-		(pin "2"
-		)
-		(pin "1"
-		)
-		(instances
-			(project "NCU"
-				(path "/3aee14c3-5480-4f7c-989e-3fef81779034/d2b1e1a0-8b64-49ff-b975-b40fa2d33dc6/70b8fb88-9c19-46a8-95e3-6c05e68e24c9"
-					(reference "JP7")
-					(unit 1)
-				)

Commit message: removed AGND and added ground garden
Connections:
- net AGND is gone; now on net GND: C33.2, C36.2, C39.2, C41.2

Commit message: added back in jumpers for internal mcu power
Parts:
- added JP6, JP7: SolderJumper_2_Bridged, Jumper:SolderJumper-2_P1.3mm_Bridged_RoundedPad1.0x1.5mm, symbol Jumper:SolderJumper_2_Bridged
Connections:
- net VCAP: now also JP7.1 (A)
- net VDDLDO: now also JP6.2 (B); no longer C34.1, L1.2
- new net 1V2_MCU: C34.1, JP6.1 (A), L1.2
- new net VFBSMPS: JP7.2 (B)
Changed lines of the file:
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@@
 	)
 	(junction
-		(at 228.6 76.2)
+		(at 31.75 38.1)
 		(diameter 0)
 		(color 0 0 0 0)
 	)
 	(junction
-		(at 31.75 38.1)
+		(at 228.6 76.2)
 		(diameter 0)
 		(color 0 0 0 0)
@@
 	)
 	(junction
-		(at 224.79 113.03)
+		(at 88.9 38.1)
 		(diameter 0)
 		(color 0 0 0 0)
 	)
 	(junction
-		(at 88.9 38.1)
+		(at 241.3 38.1)
 		(diameter 0)
 		(color 0 0 0 0)
 	)
 	(junction
-		(at 241.3 38.1)
+		(at 203.2 38.1)
 		(diameter 0)
 		(color 0 0 0 0)
 	)
 	(junction
-		(at 203.2 38.1)
+		(at 241.3 113.03)
 		(diameter 0)
 		(color 0 0 0 0)
@@
 	)
 	(junction
-		(at 254 76.2)
-		(diameter 0)
-		(color 0 0 0 0)
-	)
-	(junction
 		(at 38.1 76.2)
 		(diameter 0)
@@
 	)
 	(junction
+		(at 254 76.2)
+		(diameter 0)
+		(color 0 0 0 0)
+	)
+	(junction
 		(at 152.4 38.1)
 		(diameter 0)
@@
 	(wire
 		(pts
-			(xy 224.79 99.06) (xy 224.79 113.03)
+			(xy 234.95 125.73) (xy 241.3 125.73)
 		)
 		(stroke
@@
 	(wire
 		(pts
-			(xy 234.95 125.73) (xy 241.3 125.73)
+			(xy 38.1 48.26) (xy 38.1 50.8)
 		)
 		(stroke
@@
 	(wire
 		(pts
-			(xy 38.1 48.26) (xy 38.1 50.8)
+			(xy 241.3 38.1) (xy 260.35 38.1)
 		)
 		(stroke
@@
 	(wire
 		(pts
-			(xy 241.3 38.1) (xy 260.35 38.1)
+			(xy 241.3 113.03) (xy 228.6 113.03)
 		)
 		(stroke
@@
 	(wire
 		(pts
-			(xy 224.79 113.03) (xy 222.25 113.03)
+			(xy 222.25 113.03) (xy 228.6 113.03)
 		)
 		(stroke
@@
 	(wire
 		(pts
-			(xy 228.6 76.2) (xy 254 76.2)
-		)
-		(stroke
-			(width 0)
-			(type default)
-		)
-	)
-	(wire
-		(pts
 			(xy 260.35 38.1) (xy 266.7 38.1)
 		)
@@
 	(wire
 		(pts
+			(xy 241.3 109.22) (xy 241.3 113.03)
+		)
+		(stroke
+			(width 0)
+			(type default)
+		)
+	)
+	(wire
+		(pts
 			(xy 114.3 35.56) (xy 114.3 38.1)
 		)
@@
 	(wire
 		(pts
-			(xy 222.25 99.06) (xy 224.79 99.06)
+			(xy 222.25 99.06) (xy 241.3 99.06)
 		)
 		(stroke
@@
 	(wire
 		(pts
-			(xy 228.6 113.03) (xy 224.79 113.03)
+			(xy 195.58 76.2) (xy 208.28 76.2)
 		)
 		(stroke
@@
 	(wire
 		(pts
-			(xy 195.58 76.2) (xy 208.28 76.2)
+			(xy 266.7 88.9) (xy 260.35 88.9)
 		)
 		(stroke
@@
 	(wire
 		(pts
-			(xy 266.7 88.9) (xy 260.35 88.9)
+			(xy 266.7 86.36) (xy 266.7 88.9)
 		)
 		(stroke
@@
 	(wire
 		(pts
-			(xy 266.7 86.36) (xy 266.7 88.9)
+			(xy 63.5 76.2) (xy 63.5 78.74)
 		)
 		(stroke
@@
 	(wire
 		(pts
-			(xy 241.3 113.03) (xy 228.6 113.03)
+			(xy 63.5 48.26) (xy 63.5 50.8)
 		)
 		(stroke
@@
 	(wire
 		(pts
-			(xy 63.5 76.2) (xy 63.5 78.74)
+			(xy 208.28 76.2) (xy 214.63 76.2)
 		)
 		(stroke
@@
 	(wire
 		(pts
-			(xy 63.5 48.26) (xy 63.5 50.8)
+			(xy 101.6 38.1) (xy 114.3 38.1)
 		)
 		(stroke
@@
 	(wire
 		(pts
-			(xy 208.28 76.2) (xy 214.63 76.2)
+			(xy 76.2 73.66) (xy 76.2 76.2)
 		)
 		(stroke
@@
 	(wire
 		(pts
-			(xy 101.6 38.1) (xy 114.3 38.1)
+			(xy 38.1 76.2) (xy 63.5 76.2)
 		)
 		(stroke
@@
 	(wire
 		(pts
-			(xy 76.2 73.66) (xy 76.2 76.2)
+			(xy 152.4 38.1) (xy 165.1 38.1)
 		)
 		(stroke
@@
 	(wire
 		(pts
-			(xy 38.1 76.2) (xy 63.5 76.2)
+			(xy 260.35 88.9) (xy 260.35 91.44)
 		)
 		(stroke
@@
 	(wire
 		(pts
-			(xy 152.4 38.1) (xy 165.1 38.1)
+			(xy 245.11 76.2) (xy 254 76.2)
 		)
 		(stroke
@@
 	(wire
 		(pts
-			(xy 260.35 88.9) (xy 260.35 91.44)
+			(xy 203.2 48.26) (xy 203.2 50.8)
 		)
 		(stroke
@@
 	(wire
 		(pts
-			(xy 203.2 48.26) (xy 203.2 50.8)
+			(xy 38.1 76.2) (xy 38.1 78.74)
 		)
 		(stroke
@@
 	(wire
 		(pts
-			(xy 38.1 76.2) (xy 38.1 78.74)
+			(xy 165.1 48.26) (xy 165.1 50.8)
 		)
 		(stroke
@@
 	(wire
 		(pts
-			(xy 165.1 48.26) (xy 165.1 50.8)
+			(xy 241.3 99.06) (xy 241.3 101.6)
 		)
 		(stroke
@@
 	(wire
 		(pts
+			(xy 228.6 76.2) (xy 237.49 76.2)
+		)
+		(stroke
+			(width 0)
+			(type default)
+		)
+	)
+	(wire
+		(pts
 			(xy 222.25 76.2) (xy 228.6 76.2)
 		)
@@
 		)
 	)
+	(label "VCAP"
+		(at 241.3 113.03 0)
+		(effects
+			(font
+				(size 1.27 1.27)
+			)
+			(justify left bottom)
+		)
+	)
+	(label "VFBSD"
+		(at 241.3 99.06 0)
+		(effects
+			(font
+				(size 1.27 1.27)
+			)
+			(justify left bottom)
+		)
+	)
+	(label "VDDLDO"
+		(at 245.11 76.2 0)
+		(effects
+			(font
+				(size 1.27 1.27)
+			)
+			(justify left bottom)
+		)
+	)
+	(label "1V2_MCU"
+		(at 237.49 76.2 180)
+		(effects
+			(font
+				(size 1.27 1.27)
+			)
+			(justify right bottom)
+		)
+	)
 	(hierarchical_label "VDD"
 		(shape passive)
@@
 	)
 	(symbol
+		(lib_id "Jumper:SolderJumper_2_Bridged")
+		(at 241.3 105.41 90)
+		(unit 1)
+		(exclude_from_sim no)
+		(in_bom no)
+		(on_board yes)
+		(dnp no)
+		(property "Reference" "JP7"
+			(at 238.252 105.41 0)
+			(effects
+				(font
+					(size 1.27 1.27)
+				)
+			)
+		)
+		(property "Value" "SolderJumper_2_Bridged"
+			(at 237.49 105.41 0)
+			(effects
+				(font
+					(size 1.27 1.27)
+				)
+				(hide yes)
+			)
+		)
+		(property "Footprint" "Jumper:SolderJumper-2_P1.3mm_Bridged_RoundedPad1.0x1.5mm"
+			(at 241.3 105.41 0)
+			(effects
+				(font
+					(size 1.27 1.27)
+				)
+				(hide yes)
+			)
+		)
+		(property "Datasheet" "~"
+			(at 241.3 105.41 0)
+			(effects
+				(font
+					(size 1.27 1.27)
+				)
+				(hide yes)
+			)
+		)
+		(property "Description" "Solder Jumper, 2-pole, closed/bridged"
+			(at 241.3 105.41 0)
+			(effects
+				(font
+					(size 1.27 1.27)
+				)
+				(hide yes)
+			)
+		)
+		(pin "1"
+		)
+		(pin "2"
+		)
+		(instances
+			(project "NCU"
+				(path "/3aee14c3-5480-4f7c-989e-3fef81779034/d2b1e1a0-8b64-49ff-b975-b40fa2d33dc6/70b8fb88-9c19-46a8-95e3-6c05e68e24c9"
+					(reference "JP7")
+					(unit 1)
+				)
+			)
+		)
+	)
+	(symbol
 		(lib_id "Device:C")
 		(at 266.7 82.55 0)
@@
 					(unit 1)
 				)
+			)
+		)
+	)
+	(symbol
+		(lib_id "Jumper:SolderJumper_2_Bridged")
+		(at 241.3 76.2 0)
+		(unit 1)
+		(exclude_from_sim no)
+		(in_bom no)
+		(on_board yes)
+		(dnp no)
+		(property "Reference" "JP6"
+			(at 241.3 73.152 0)
+			(effects
+				(font
+					(size 1.27 1.27)
+				)
+			)
+		)
+		(property "Value" "SolderJumper_2_Bridged"
+			(at 241.3 72.39 0)
+			(effects
+				(font
+					(size 1.27 1.27)
+				)
+				(hide yes)
+			)
+		)
+		(property "Footprint" "Jumper:SolderJumper-2_P1.3mm_Bridged_RoundedPad1.0x1.5mm"
+			(at 241.3 76.2 0)
+			(effects
+				(font
+					(size 1.27 1.27)
+				)
+				(hide yes)
+			)
+		)
+		(property "Datasheet" "~"
+			(at 241.3 76.2 0)
+			(effects
+				(font
+					(size 1.27 1.27)
+				)
+				(hide yes)
+			)
+		)
+		(property "Description" "Solder Jumper, 2-pole, closed/bridged"
+			(at 241.3 76.2 0)
+			(effects
+				(font
+					(size 1.27 1.27)
+				)
+				(hide yes)
+			)
+		)
+		(pin "1"
+		)
+		(pin "2"
+		)
+		(instances
+			(project ""
+				(path "/3aee14c3-5480-4f7c-989e-3fef81779034/d2b1e1a0-8b64-49ff-b975-b40fa2d33dc6/70b8fb88-9c19-46a8-95e3-6c05e68e24c9"
+					(reference "JP6")
+					(unit 1)
+				)

Commit message: added jumper for VCAP connection to 1V2MCU. Fixed resistors on ethernet IF
Parts:
- added JP8: SolderJumper_2_Open, Jumper:SolderJumper-2_P1.3mm_Open_RoundedPad1.0x1.5mm, symbol Jumper:SolderJumper_2_Open
Connections:
- net 1V2_MCU: now also JP8.2 (B)
- net VCAP: now also JP8.1 (A)
Other:
- moved on the sheet: C35, C37, JP7

Commit message: updates from bom release
Parts:
- C13: value 4.7uF -> 4.7u
- C14, C15, C16, C18, C19, C20, C21, C23, C25, C26, C27, C28, C29, C30, C31, C36, C38, C40, C41: value 100nF -> 100n
- C17, C33, C39: value 1uF -> 1u
- C22, C24, C34: value 10uF -> 10u
- C32: value 220pF -> 220p
- C35, C37: value 2.2uF -> 2.2u
- L1: value 2.2uH -> 2.2u
Changed lines of the file:
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@@
 			)
 		)
-		(property "Value" "100nF"
+		(property "Value" "100n"
 			(at 167.64 45.72 0)
 			(effects
@@
 			)
 		)
-		(property "Value" "10uF"
+		(property "Value" "10u"
 			(at 104.14 83.82 0)
 			(effects
@@
 			)
 		)
-		(property "Value" "100nF"
+		(property "Value" "100n"
 			(at 243.84 45.72 0)
 			(effects
@@
 			)
 		)
-		(property "Value" "100nF"
+		(property "Value" "100n"
 			(at 275.59 45.72 0)
 			(effects
@@
 			)
 		)
-		(property "Value" "100nF"
+		(property "Value" "100n"
 			(at 205.74 45.72 0)
 			(effects
@@
 			)
 		)
-		(property "Value" "1uF"
+		(property "Value" "1u"
 			(at 262.89 45.72 0)
 			(effects
@@
 			)
 		)
-		(property "Value" "100nF"
+		(property "Value" "100n"
 			(at 129.54 45.72 0)
 			(effects
@@
 			)
 		)
-		(property "Value" "10uF"
+		(property "Value" "10u"
 			(at 231.14 83.82 0)
 			(effects
@@
 			)
 		)
-		(property "Value" "100nF"
+		(property "Value" "100n"
 			(at 269.24 83.82 0)
 			(effects
@@
 			)
 		)
-		(property "Value" "100nF"
+		(property "Value" "100n"
 			(at 78.74 83.82 0)
 			(effects
@@
 			)
 		)
-		(property "Value" "100nF"
+		(property "Value" "100n"
 			(at 193.04 45.72 0)
 			(effects
@@
 			)
 		)
-		(property "Value" "10uF"
+		(property "Value" "10u"
 			(at 116.84 83.82 0)
 			(effects
@@
 			)
 		)
-		(property "Value" "1uF"
+		(property "Value" "1u"
 			(at 231.14 45.72 0)
 			(effects
@@
 			)
 		)
-		(property "Value" "100nF"
+		(property "Value" "100n"
 			(at 66.04 45.72 0)
 			(effects
@@
 			)
 		)
-		(property "Value" "100nF"
+		(property "Value" "100n"
 			(at 116.84 45.72 0)
 			(effects
@@
 			)
 		)
-		(property "Value" "100nF"
+		(property "Value" "100n"
 			(at 91.44 45.72 0)
 			(effects
@@
 			)
 		)
-		(property "Value" "100nF"
+		(property "Value" "100n"
 			(at 78.74 45.72 0)
 			(effects
@@
 			)
 		)
-		(property "Value" "2.2uF"
+		(property "Value" "2.2u"
 			(at 213.36 120.65 0)
 			(effects
@@
 			)
 		)
-		(property "Value" "100nF"
+		(property "Value" "100n"
 			(at 53.34 45.72 0)
 			(effects
@@
 			)
 		)
-		(property "Value" "1uF"
+		(property "Value" "1u"
 			(at 66.04 83.82 0)
 			(effects
@@
 			)
 		)
-		(property "Value" "2.2uH"
+		(property "Value" "2.2u"
 			(at 218.44 73.66 90)
 			(effects
@@
 			)
 		)
-		(property "Value" "100nF"
+		(property "Value" "100n"
 			(at 180.34 45.72 0)
 			(effects
@@
 			)
 		)
-		(property "Value" "100nF"
+		(property "Value" "100n"
 			(at 40.64 83.82 0)
 			(effects
@@
 			)
 		)
-		(property "Value" "100nF"
+		(property "Value" "100n"
 			(at 154.94 45.72 0)
 			(effects
@@
 			)
 		)
-		(property "Value" "2.2uF"
+		(property "Value" "2.2u"
 			(at 226.06 120.65 0)
 			(effects
@@
 			)
 		)
-		(property "Value" "4.7uF"
+		(property "Value" "4.7u"
 			(at 40.64 45.72 0)
 			(effects
@@
 			)
 		)
-		(property "Value" "100nF"
+		(property "Value" "100n"
 			(at 104.14 45.72 0)
 			(effects
@@
 			)
 		)
-		(property "Value" "100nF"
+		(property "Value" "100n"
 			(at 142.24 45.72 0)
 			(effects
@@
 			)
 		)
-		(property "Value" "220pF"
+		(property "Value" "220p"
 			(at 210.82 83.82 0)
 			(effects
@@
 			)
 		)
-		(property "Value" "100nF"
+		(property "Value" "100n"
 			(at 256.54 83.82 0)
 			(effects
