File: pcb/PWR.kicad_sch (KiCad schematic)
At the start: 6 parts

Commit message: power done
Parts:
- added A5V_PG, LV_PG, TP3, USB_PWR_ST: LV_5V, TestPoint:TestPoint_THTPad_D2.0mm_Drill1.0mm, symbol Connector:TestPoint
- added TP2: 12V, TestPoint:TestPoint_THTPad_D2.0mm_Drill1.0mm, symbol Connector:TestPoint
- added TP4: USB_5V, TestPoint:TestPoint_THTPad_D2.0mm_Drill1.0mm, symbol Connector:TestPoint
- added TP5: 5V, TestPoint:TestPoint_THTPad_D2.0mm_Drill1.0mm, symbol Connector:TestPoint
- added TP6: A5V, TestPoint:TestPoint_THTPad_D2.0mm_Drill1.0mm, symbol Connector:TestPoint
- added TP7: AGND, TestPoint:TestPoint_THTPad_D2.0mm_Drill1.0mm, symbol Connector:TestPoint
- added TP8: 3V3, TestPoint:TestPoint_THTPad_D2.0mm_Drill1.0mm, symbol Connector:TestPoint
- added TP9: 3V3_PG, TestPoint:TestPoint_THTPad_D2.0mm_Drill1.0mm, symbol Connector:TestPoint
- TP1: value TestPoint -> GND
Connections:
- net 12V: no longer R5.1
- net 3V3: now also TP8.1
- net 3V3_PG: now also TP9.1
- net 5V: now also TP5.1
- net A5V: now also TP6.1
- net A5V_PG: now also A5V_PG.1
- net AGND: now also TP7.1
- net GND: now also TP1.1
- net LV_PG: now also LV_PG.1
- net PWR_LV_5V/LV_5V: now also TP3.1
- net USB_5V: now also TP4.1
- net USB_PWR_ST: now also USB_PWR_ST.1
- new net 12V_PRT: R5.1, TP2.1
Other:
- added sheet PWR_PRT (PWR_PRT.kicad_sch)
- moved on the sheet: D1, D2, NT1, R5, R6, TP1

Commit message: reannotated, updated some symbols
Parts:
- renumbered A5V_PG to A5V_PG1, LV_PG to LV_PG1, R5 to R1, R6 to R2, TP2 to TP1, TP1 to TP2, TP6 to TP4, TP7 to TP5, TP4 to TP6, TP9 to TP7, TP5 to TP8, TP8 to TP9, USB_PWR_ST to USB_PWR_ST1

Commit message: all power supplies laid out I think
Parts:
- removed A5V_PG1, LV_PG1, USB_PWR_ST1: LV_5V, TestPoint:TestPoint_THTPad_D2.0mm_Drill1.0mm, symbol Connector:TestPoint
- removed TP7: 3V3_PG, TestPoint:TestPoint_THTPad_D2.0mm_Drill1.0mm, symbol Connector:TestPoint

Commit message: removed AGND and added ground garden
Parts:
- removed NT1: NetTie_2, NetTie:NetTie-2_SMD_Pad0.5mm, symbol Device:NetTie_2
- removed TP5: AGND, TestPoint:TestPoint_THTPad_D2.0mm_Drill1.0mm, symbol Connector:TestPoint

Commit message: added 10k resistor to USB VBUS line
Other:
- sheet PWR_A5V ports: added none; removed AGND
Changed lines of the file:
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@@
-			)
-		)
-		(pin "AGND" passive
-			(at 107.95 91.44 0)
-			(effects
-				(font
-					(size 1.27 1.27)
-				)
-				(justify right)
 			)
 		)

Commit message: updates from bom release
Parts:
- R2: value 260R -> 620
Changed lines of the file:
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@@
 			)
 		)
-		(property "Value" "260R"
+		(property "Value" "620"
 			(at 42.418 102.616 0)
 			(effects
