File: pcb/PWR_3V3.kicad_sch (KiCad schematic)
At the start: 12 parts, among them IC5 TPS628101HQWRWYRQ1

Commit message: power done
Parts:
- C78: value 22uF -> 10uF
- L3: footprint INDPM7066X240N -> SamacSys_Parts:XFL4012
Changed lines of the file:
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@@
-	)
-	(junction
-		(at 114.3 81.28)
-		(diameter 0)
-		(color 0 0 0 0)
-	)
-	(junction
-		(at 120.65 81.28)
-		(diameter 0)
-		(color 0 0 0 0)
 	)
 	(junction
@@
 	(wire
 		(pts
-			(xy 139.7 81.28) (xy 139.7 80.01)
-		)
-		(stroke
-			(width 0)
-			(type default)
-		)
-	)
-	(wire
-		(pts
 			(xy 88.9 80.01) (xy 88.9 81.28)
 		)
@@
 	(wire
 		(pts
-			(xy 114.3 81.28) (xy 120.65 81.28)
-		)
-		(stroke
-			(width 0)
-			(type default)
-		)
-	)
-	(wire
-		(pts
 			(xy 146.05 60.96) (xy 146.05 62.23)
 		)
@@
 	(wire
 		(pts
-			(xy 120.65 80.01) (xy 120.65 81.28)
-		)
-		(stroke
-			(width 0)
-			(type default)
-		)
-	)
-	(wire
-		(pts
 			(xy 36.83 58.42) (xy 39.37 58.42)
 		)
@@
 	(wire
 		(pts
-			(xy 139.7 81.28) (xy 120.65 81.28)
+			(xy 120.65 80.01) (xy 120.65 83.82)
 		)
 		(stroke
@@
 		(pts
 			(xy 184.15 69.85) (xy 184.15 71.12)
+		)
+		(stroke
+			(width 0)
+			(type default)
+		)
+	)
+	(wire
+		(pts
+			(xy 139.7 80.01) (xy 139.7 83.82)
 		)
 		(stroke
@@
 			)
 		)
-		(property "Value" "22uF"
+		(property "Value" "10uF"
 			(at 187.198 67.31 0)
 			(effects
@@
 			)
 		)
-		(property "Footprint" "INDPM7066X240N"
+		(property "Footprint" "SamacSys_Parts:XFL4012"
 			(at 127 60.96 0)
 			(effects
@@
 				(path "/3aee14c3-5480-4f7c-989e-3fef81779034/05e3be97-98f6-4518-a1a7-240d4da327e6/c5136008-5582-44d5-9c96-36b624677ffa"
 					(reference "#PWR0278")
+					(unit 1)
+				)
+			)
+		)
+	)
+	(symbol
+		(lib_id "power:GND")
+		(at 120.65 83.82 0)
+		(unit 1)
+		(exclude_from_sim no)
+		(in_bom yes)
+		(on_board yes)
+		(dnp no)
+		(property "Reference" "#PWR0344"
+			(at 120.65 90.17 0)
+			(effects
+				(font
+					(size 1.27 1.27)
+				)
+				(hide yes)
+			)
+		)
+		(property "Value" "GND"
+			(at 120.65 87.63 0)
+			(effects
+				(font
+					(size 1.27 1.27)
+				)
+			)
+		)
+		(property "Footprint" ""
+			(at 120.65 83.82 0)
+			(effects
+				(font
+					(size 1.27 1.27)
+				)
+				(hide yes)
+			)
+		)
+		(property "Datasheet" ""
+			(at 120.65 83.82 0)
+			(effects
+				(font
+					(size 1.27 1.27)
+				)
+				(hide yes)
+			)
+		)
+		(property "Description" "Power symbol creates a global label with name \"GND\" , ground"
+			(at 120.65 83.82 0)
+			(effects
+				(font
+					(size 1.27 1.27)
+				)
+				(hide yes)
+			)
+		)
+		(pin "1"
+		)
+		(instances
+			(project "NCU"
+				(path "/3aee14c3-5480-4f7c-989e-3fef81779034/05e3be97-98f6-4518-a1a7-240d4da327e6/c5136008-5582-44d5-9c96-36b624677ffa"
+					(reference "#PWR0344")
 					(unit 1)
 				)
@@
 					(unit 1)
 				)
+			)
+		)
+	)
+	(symbol
+		(lib_id "power:GND")
+		(at 139.7 83.82 0)
+		(unit 1)
+		(exclude_from_sim no)
+		(in_bom yes)
+		(on_board yes)
+		(dnp no)
+		(property "Reference" "#PWR0345"
+			(at 139.7 90.17 0)
+			(effects
+				(font
+					(size 1.27 1.27)
+				)
+				(hide yes)
+			)
+		)
+		(property "Value" "GND"
+			(at 139.7 87.63 0)
+			(effects
+				(font
+					(size 1.27 1.27)
+				)
+			)
+		)
+		(property "Footprint" ""
+			(at 139.7 83.82 0)
+			(effects
+				(font
+					(size 1.27 1.27)
+				)
+				(hide yes)
+			)
+		)
+		(property "Datasheet" ""
+			(at 139.7 83.82 0)
+			(effects
+				(font
+					(size 1.27 1.27)
+				)
+				(hide yes)
+			)
+		)
+		(property "Description" "Power symbol creates a global label with name \"GND\" , ground"
+			(at 139.7 83.82 0)
+			(effects
+				(font
+					(size 1.27 1.27)
+				)
+				(hide yes)
+			)
+		)
+		(pin "1"
+		)
+		(instances
+			(project "NCU"
+				(path "/3aee14c3-5480-4f7c-989e-3fef81779034/05e3be97-98f6-4518-a1a7-240d4da327e6/c5136008-5582-44d5-9c96-36b624677ffa"
+					(reference "#PWR0345")
+					(unit 1)
+				)

Commit message: reannotated, updated some symbols
Parts:
- renumbered C73 to C80, C74 to C81, C75 to C82, C76 to C83, C77 to C84, C78 to C85, IC5 to IC7, R77 to R114, R78 to R115, R79 to R116, R80 to R117
Changed lines of the file:
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@@
 		(dnp no)
 		(fields_autoplaced yes)
-		(property "Reference" "R80"
+		(property "Reference" "R117"
 			(at 142.24 74.9299 0)
 			(effects
@@
 			(project "NCU"
 				(path "/3aee14c3-5480-4f7c-989e-3fef81779034/05e3be97-98f6-4518-a1a7-240d4da327e6/c5136008-5582-44d5-9c96-36b624677ffa"
-					(reference "R80")
+					(reference "R117")
 					(unit 1)
 				)
@@
 		(on_board yes)
 		(dnp no)
-		(property "Reference" "R77"
+		(property "Reference" "R114"
 			(at 40.64 46.228 0)
 			(effects
@@
 			(project "NCU"
 				(path "/3aee14c3-5480-4f7c-989e-3fef81779034/05e3be97-98f6-4518-a1a7-240d4da327e6/c5136008-5582-44d5-9c96-36b624677ffa"
-					(reference "R77")
+					(reference "R114")
 					(unit 1)
 				)
@@
 		(on_board yes)
 		(dnp no)
-		(property "Reference" "#PWR0276"
+		(property "Reference" "#PWR0370"
 			(at 21.59 33.02 0)
 			(effects
@@
 			(project "NCU"
 				(path "/3aee14c3-5480-4f7c-989e-3fef81779034/05e3be97-98f6-4518-a1a7-240d4da327e6/c5136008-5582-44d5-9c96-36b624677ffa"
-					(reference "#PWR0276")
+					(reference "#PWR0370")
 					(unit 1)
 				)
@@
 		(on_board yes)
 		(dnp no)
-		(property "Reference" "#PWR0280"
+		(property "Reference" "#PWR0374"
 			(at 88.9 88.9 0)
 			(effects
@@
 			(project "NCU"
 				(path "/3aee14c3-5480-4f7c-989e-3fef81779034/05e3be97-98f6-4518-a1a7-240d4da327e6/c5136008-5582-44d5-9c96-36b624677ffa"
-					(reference "#PWR0280")
+					(reference "#PWR0374")
 					(unit 1)
 				)
@@
 		(on_board yes)
 		(dnp no)
-		(property "Reference" "#PWR0283"
+		(property "Reference" "#PWR0379"
 			(at 184.15 63.5 0)
 			(effects
@@
 			(project "NCU"
 				(path "/3aee14c3-5480-4f7c-989e-3fef81779034/05e3be97-98f6-4518-a1a7-240d4da327e6/c5136008-5582-44d5-9c96-36b624677ffa"
-					(reference "#PWR0283")
+					(reference "#PWR0379")
 					(unit 1)
 				)
@@
 		(on_board yes)
 		(dnp no)
-		(property "Reference" "#PWR0277"
+		(property "Reference" "#PWR0371"
 			(at 24.13 45.72 0)
 			(effects
@@
 			(project "NCU"
 				(path "/3aee14c3-5480-4f7c-989e-3fef81779034/05e3be97-98f6-4518-a1a7-240d4da327e6/c5136008-5582-44d5-9c96-36b624677ffa"
-					(reference "#PWR0277")
+					(reference "#PWR0371")
 					(unit 1)
 				)
@@
 		(dnp no)
 		(fields_autoplaced yes)
-		(property "Reference" "R78"
+		(property "Reference" "R115"
 			(at 91.44 74.9299 0)
 			(effects
@@
 			(project "NCU"
 				(path "/3aee14c3-5480-4f7c-989e-3fef81779034/05e3be97-98f6-4518-a1a7-240d4da327e6/c5136008-5582-44d5-9c96-36b624677ffa"
-					(reference "R78")
+					(reference "R115")
 					(unit 1)
 				)
@@
 		(on_board yes)
 		(dnp no)
-		(property "Reference" "C78"
+		(property "Reference" "C85"
 			(at 187.452 64.77 0)
 			(effects
@@
 			(project "NCU"
 				(path "/3aee14c3-5480-4f7c-989e-3fef81779034/05e3be97-98f6-4518-a1a7-240d4da327e6/c5136008-5582-44d5-9c96-36b624677ffa"
-					(reference "C78")
+					(reference "C85")
 					(unit 1)
 				)
@@
 		(on_board yes)
 		(dnp no)
-		(property "Reference" "#PWR0282"
+		(property "Reference" "#PWR0378"
 			(at 158.75 78.74 0)
 			(effects
@@
 			(project "NCU"
 				(path "/3aee14c3-5480-4f7c-989e-3fef81779034/05e3be97-98f6-4518-a1a7-240d4da327e6/c5136008-5582-44d5-9c96-36b624677ffa"
-					(reference "#PWR0282")
+					(reference "#PWR0378")
 					(unit 1)
 				)
@@
 		(on_board yes)
 		(dnp no)
-		(property "Reference" "C77"
+		(property "Reference" "C84"
 			(at 174.752 64.77 0)
 			(effects
@@
 			(project "NCU"
 				(path "/3aee14c3-5480-4f7c-989e-3fef81779034/05e3be97-98f6-4518-a1a7-240d4da327e6/c5136008-5582-44d5-9c96-36b624677ffa"
-					(reference "C77")
+					(reference "C84")
 					(unit 1)
 				)
@@
 		(on_board yes)
 		(dnp no)
-		(property "Reference" "#PWR0278"
+		(property "Reference" "#PWR0372"
 			(at 30.48 24.13 0)
 			(effects
@@
 			(project "NCU"
 				(path "/3aee14c3-5480-4f7c-989e-3fef81779034/05e3be97-98f6-4518-a1a7-240d4da327e6/c5136008-5582-44d5-9c96-36b624677ffa"
-					(reference "#PWR0278")
+					(reference "#PWR0372")
 					(unit 1)
 				)
@@
 		(on_board yes)
 		(dnp no)
-		(property "Reference" "#PWR0344"
+		(property "Reference" "#PWR0376"
 			(at 120.65 90.17 0)
 			(effects
@@
 			(project "NCU"
 				(path "/3aee14c3-5480-4f7c-989e-3fef81779034/05e3be97-98f6-4518-a1a7-240d4da327e6/c5136008-5582-44d5-9c96-36b624677ffa"
-					(reference "#PWR0344")
+					(reference "#PWR0376")
 					(unit 1)
 				)
@@
 		(dnp no)
 		(fields_autoplaced yes)
-		(property "Reference" "IC5"
+		(property "Reference" "IC7"
 			(at 63.5 48.26 0)
 			(effects
@@
 			(project "NCU"
 				(path "/3aee14c3-5480-4f7c-989e-3fef81779034/05e3be97-98f6-4518-a1a7-240d4da327e6/c5136008-5582-44d5-9c96-36b624677ffa"
-					(reference "IC5")
+					(reference "IC7")
 					(unit 1)
 				)
@@
 		(dnp no)
 		(fields_autoplaced yes)
-		(property "Reference" "R79"
+		(property "Reference" "R116"
 			(at 135.89 64.7699 0)
 			(effects
@@
 			(project "NCU"
 				(path "/3aee14c3-5480-4f7c-989e-3fef81779034/05e3be97-98f6-4518-a1a7-240d4da327e6/c5136008-5582-44d5-9c96-36b624677ffa"
-					(reference "R79")
+					(reference "R116")
 					(unit 1)
 				)
@@
 		(on_board yes)
 		(dnp no)
-		(property "Reference" "#PWR0281"
+		(property "Reference" "#PWR0375"
 			(at 120.65 58.42 0)
 			(effects
@@
 			(project "NCU"
 				(path "/3aee14c3-5480-4f7c-989e-3fef81779034/05e3be97-98f6-4518-a1a7-240d4da327e6/c5136008-5582-44d5-9c96-36b624677ffa"
-					(reference "#PWR0281")
+					(reference "#PWR0375")
 					(unit 1)
 				)
@@
 		(on_board yes)
 		(dnp no)
-		(property "Reference" "#PWR0275"
+		(property "Reference" "#PWR0369"
 			(at 21.59 24.13 0)
 			(effects
@@
 			(project "NCU"
 				(path "/3aee14c3-5480-4f7c-989e-3fef81779034/05e3be97-98f6-4518-a1a7-240d4da327e6/c5136008-5582-44d5-9c96-36b624677ffa"
-					(reference "#PWR0275")
+					(reference "#PWR0369")
 					(unit 1)
 				)
@@
 		(on_board yes)
 		(dnp no)
-		(property "Reference" "C75"
+		(property "Reference" "C82"
 			(at 149.352 64.77 0)
 			(effects
@@
 			(project "NCU"
 				(path "/3aee14c3-5480-4f7c-989e-3fef81779034/05e3be97-98f6-4518-a1a7-240d4da327e6/c5136008-5582-44d5-9c96-36b624677ffa"
-					(reference "C75")
+					(reference "C82")
 					(unit 1)
 				)
@@
 		(on_board yes)
 		(dnp no)
-		(property "Reference" "C74"
+		(property "Reference" "C81"
 			(at 123.952 74.93 0)
 			(effects
@@
 			(project "NCU"
 				(path "/3aee14c3-5480-4f7c-989e-3fef81779034/05e3be97-98f6-4518-a1a7-240d4da327e6/c5136008-5582-44d5-9c96-36b624677ffa"
-					(reference "C74")
+					(reference "C81")
 					(unit 1)
 				)
@@
 		(on_board yes)
 		(dnp no)
-		(property "Reference" "C73"
+		(property "Reference" "C80"
 			(at 104.902 74.93 0)
 			(effects
@@
 			(project "NCU"
 				(path "/3aee14c3-5480-4f7c-989e-3fef81779034/05e3be97-98f6-4518-a1a7-240d4da327e6/c5136008-5582-44d5-9c96-36b624677ffa"
-					(reference "C73")
+					(reference "C80")
 					(unit 1)
 				)
@@
 		(on_board yes)
 		(dnp no)
-		(property "Reference" "#PWR0279"
+		(property "Reference" "#PWR0373"
 			(at 36.83 45.72 0)
 			(effects
@@
 			(project "NCU"
 				(path "/3aee14c3-5480-4f7c-989e-3fef81779034/05e3be97-98f6-4518-a1a7-240d4da327e6/c5136008-5582-44d5-9c96-36b624677ffa"
-					(reference "#PWR0279")
+					(reference "#PWR0373")
 					(unit 1)
 				)
@@
 		(on_board yes)
 		(dnp no)
-		(property "Reference" "C76"
+		(property "Reference" "C83"
 			(at 162.052 64.77 0)
 			(effects
@@
 			(project "NCU"
 				(path "/3aee14c3-5480-4f7c-989e-3fef81779034/05e3be97-98f6-4518-a1a7-240d4da327e6/c5136008-5582-44d5-9c96-36b624677ffa"
-					(reference "C76")
+					(reference "C83")
 					(unit 1)
 				)
@@
 		(on_board yes)
 		(dnp no)
-		(property "Reference" "#PWR0345"
+		(property "Reference" "#PWR0377"
 			(at 139.7 90.17 0)
 			(effects
@@
 			(project "NCU"
 				(path "/3aee14c3-5480-4f7c-989e-3fef81779034/05e3be97-98f6-4518-a1a7-240d4da327e6/c5136008-5582-44d5-9c96-36b624677ffa"
-					(reference "#PWR0345")
-					(unit 1)
-				)
+					(reference "#PWR0377")
+					(unit 1)
+				)

Commit message: updates from bom release
Parts:
- C80: value 4.7nF -> 4.7n
- C81, C83, C84: value 22uF -> 22u
- C82: value 10pF -> 10p
- C85: value 10uF -> 10u
- L3: value 0.47uH -> 0.47u
Changed lines of the file:
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@@
 			)
 		)
-		(property "Value" "10uF"
+		(property "Value" "10u"
 			(at 187.198 67.31 0)
 			(effects
@@
 			)
 		)
-		(property "Value" "0.47uH"
+		(property "Value" "0.47u"
 			(at 127 58.42 90)
 			(effects
@@
 			)
 		)
-		(property "Value" "22uF"
+		(property "Value" "22u"
 			(at 174.498 67.31 0)
 			(effects
@@
 			)
 		)
-		(property "Value" "10pF"
+		(property "Value" "10p"
 			(at 149.098 67.31 0)
 			(effects
@@
 			)
 		)
-		(property "Value" "22uF"
+		(property "Value" "22u"
 			(at 123.698 77.47 0)
 			(effects
@@
 			)
 		)
-		(property "Value" "4.7nF"
+		(property "Value" "4.7n"
 			(at 104.648 77.47 0)
 			(effects
@@
 			)
 		)
-		(property "Value" "22uF"
+		(property "Value" "22u"
 			(at 161.798 67.31 0)
 			(effects

Commit message: updated to match board changes
Parts:
- R116: value 88.7k -> 0
- R117: now not fitted
Changed lines of the file:
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@@
 		(in_bom yes)
 		(on_board yes)
-		(dnp no)
+		(dnp yes)
 		(fields_autoplaced yes)
 		(property "Reference" "R117"
@@
 			)
 		)
-		(property "Value" "88.7k"
+		(property "Value" "0"
 			(at 135.89 67.3099 0)
 			(effects
